File: nlp-16a/Hardware/A_B_BUS_Ctrl/A_B_BUS_Ctrl/decoder.kicad_sch (KiCad schematic)
At the start: 6 parts

Commit message: 配線作業開始
Parts:
- U24, U32, U40: renamed from U?; footprint (none) -> Package_DIP:DIP-14_W7.62mm
Connections:
- net A: now also U40.4; no longer U40.1
- net B: now also U40.5; no longer U40.2
- net C: now also U32.4; no longer U32.10
- net D: now also U24.4; no longer U24.10
- net INTERNAL: now also U24.10; no longer U24.13
- net OUT: now also U24.8; no longer U24.11
- new net: U40.10, U40.6, U40.9
- new net: U32.5, U40.8
- new net: U24.6, U24.9
- new net: U24.5, U32.8
- new net: U32.10, U32.6, U32.9
Changed lines of the file:
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@@
     (effects (font (size 1.27 1.27)) (justify right))
   )
-  (symbol (lib_id "CD74HCXX:CD74HC00") (at 81.28 67.31 0) (unit 1)
+  (symbol (lib_id "CD74HCXX:CD74HC00") (at 81.28 67.31 0) (unit 2)
     (in_bom yes) (on_board yes) (fields_autoplaced)
-    (property "Reference" "U?" (id 0) (at 81.28 58.42 0))
+    (property "Reference" "U40" (id 0) (at 81.28 58.42 0))
     (property "Value" "CD74HC00" (id 1) (at 81.28 60.96 0))
-    (property "Footprint" "" (id 2) (at 76.2 67.31 0))
+    (property "Footprint" "Package_DIP:DIP-14_W7.62mm" (id 2) (at 76.2 67.31 0)
+      (effects (font (size 1.27 1.27)) hide)
+    )
     (property "Datasheet" "" (id 3) (at 76.2 67.31 0))
     (pin "14")
@@
     (pin "13")
   )
-  (symbol (lib_id "CD74HCXX:CD74HC00") (at 99.06 67.31 0) (unit 2)
+  (symbol (lib_id "CD74HCXX:CD74HC00") (at 99.06 67.31 0) (unit 3)
     (in_bom yes) (on_board yes) (fields_autoplaced)
-    (property "Reference" "U?" (id 0) (at 99.06 58.42 0))
+    (property "Reference" "U40" (id 0) (at 99.06 58.42 0))
     (property "Value" "CD74HC00" (id 1) (at 99.06 60.96 0))
-    (property "Footprint" "" (id 2) (at 93.98 67.31 0))
+    (property "Footprint" "Package_DIP:DIP-14_W7.62mm" (id 2) (at 93.98 67.31 0)
+      (effects (font (size 1.27 1.27)) hide)
+    )
     (property "Datasheet" "" (id 3) (at 93.98 67.31 0))
     (pin "14")
@@
     (pin "13")
   )
-  (symbol (lib_id "CD74HCXX:CD74HC00") (at 177.8 67.31 0) (unit 4)
+  (symbol (lib_id "CD74HCXX:CD74HC00") (at 177.8 67.31 0) (unit 3)
     (in_bom yes) (on_board yes) (fields_autoplaced)
-    (property "Reference" "U?" (id 0) (at 177.8 58.42 0))
+    (property "Reference" "U24" (id 0) (at 177.8 58.42 0))
     (property "Value" "CD74HC00" (id 1) (at 177.8 60.96 0))
-    (property "Footprint" "" (id 2) (at 172.72 67.31 0))
+    (property "Footprint" "Package_DIP:DIP-14_W7.62mm" (id 2) (at 172.72 67.31 0)
+      (effects (font (size 1.27 1.27)) hide)
+    )
     (property "Datasheet" "" (id 3) (at 172.72 67.31 0))
     (pin "14")
@@
     (pin "13")
   )
-  (symbol (lib_id "CD74HCXX:CD74HC00") (at 157.48 67.31 0) (unit 3)
+  (symbol (lib_id "CD74HCXX:CD74HC00") (at 157.48 67.31 0) (mirror x) (unit 2)
     (in_bom yes) (on_board yes) (fields_autoplaced)
-    (property "Reference" "U?" (id 0) (at 157.48 58.42 0))
+    (property "Reference" "U24" (id 0) (at 157.48 58.42 0))
     (property "Value" "CD74HC00" (id 1) (at 157.48 60.96 0))
-    (property "Footprint" "" (id 2) (at 152.4 67.31 0))
+    (property "Footprint" "Package_DIP:DIP-14_W7.62mm" (id 2) (at 152.4 67.31 0)
+      (effects (font (size 1.27 1.27)) hide)
+    )
     (property "Datasheet" "" (id 3) (at 152.4 67.31 0))
     (pin "14")
@@
     (pin "13")
   )
-  (symbol (lib_id "CD74HCXX:CD74HC00") (at 119.38 67.31 0) (unit 3)
+  (symbol (lib_id "CD74HCXX:CD74HC00") (at 119.38 67.31 0) (mirror x) (unit 2)
     (in_bom yes) (on_board yes) (fields_autoplaced)
-    (property "Reference" "U?" (id 0) (at 119.38 58.42 0))
+    (property "Reference" "U32" (id 0) (at 119.38 58.42 0))
     (property "Value" "CD74HC00" (id 1) (at 119.38 60.96 0))
-    (property "Footprint" "" (id 2) (at 114.3 67.31 0))
+    (property "Footprint" "Package_DIP:DIP-14_W7.62mm" (id 2) (at 114.3 67.31 0)
+      (effects (font (size 1.27 1.27)) hide)
+    )
     (property "Datasheet" "" (id 3) (at 114.3 67.31 0))
     (pin "14")
@@
     (pin "13")
   )
-  (symbol (lib_id "CD74HCXX:CD74HC00") (at 137.16 67.31 0) (unit 4)
+  (symbol (lib_id "CD74HCXX:CD74HC00") (at 137.16 67.31 0) (unit 3)
     (in_bom yes) (on_board yes) (fields_autoplaced)
-    (property "Reference" "U?" (id 0) (at 137.16 58.42 0))
+    (property "Reference" "U32" (id 0) (at 137.16 58.42 0))
     (property "Value" "CD74HC00" (id 1) (at 137.16 60.96 0))
-    (property "Footprint" "" (id 2) (at 132.08 67.31 0))
+    (property "Footprint" "Package_DIP:DIP-14_W7.62mm" (id 2) (at 132.08 67.31 0)
+      (effects (font (size 1.27 1.27)) hide)
+    )
     (property "Datasheet" "" (id 3) (at 132.08 67.31 0))
     (pin "14")
