File: nlp-16a/Hardware/A_B_BUS_Ctrl/A_B_BUS_Ctrl/BUS_OUTPUT_Correction.kicad_sch (KiCad schematic)
At the start: 0 parts

Commit message: 信号補正部追加
Other:
- added sheet Correction0 (Correction.kicad_sch)
- added sheet Correction1 (Correction.kicad_sch)
- added sheet Correction10 (Correction.kicad_sch)
- added sheet Correction11 (Correction.kicad_sch)
- added sheet Correction12 (Correction.kicad_sch)
- added sheet Correction13 (Correction.kicad_sch)
- added sheet Correction14 (Correction.kicad_sch)
- added sheet Correction15 (Correction.kicad_sch)
- added sheet Correction2 (Correction.kicad_sch)
- added sheet Correction3 (Correction.kicad_sch)
- added sheet Correction4 (Correction.kicad_sch)
- added sheet Correction5 (Correction.kicad_sch)
- added sheet Correction6 (Correction.kicad_sch)
- added sheet Correction7 (Correction.kicad_sch)
- added sheet Correction8 (Correction.kicad_sch)
- added sheet Correction9 (Correction.kicad_sch)
- note added: "信号補正部 Regデータバスから送られてくる生のデータ(RAW_DATA)は選択されたレジスタの位置によって反転，非反転が異なる． 従って選択されたレジスタの物理的な位置を検出し，適切に補正する必要がある． 補正はレジスタ部から送られてくる補正信号を基に反転，非反転を制御し，すべてのビットに対して適切に反転，非反転の処理を加えALUへデータを送る"

Commit message: 配線作業開始
Parts:
- added U43: CD74HC00, Package_DIP:DIP-14_W7.62mm, symbol CD74HCXX:CD74HC00
Connections:
- net Correction: now also U43.1
- new net Correction0/Correction: U43.3
- new net GND: U43.10, U43.12, U43.13, U43.4, U43.5, U43.7 (GND), U43.7 (GND), U43.7 (GND), U43.7 (GND), U43.9
- new net VCC: U43.14 (VCC), U43.14 (VCC), U43.14 (VCC), U43.14 (VCC), U43.2
- no-connect marks 0 -> 3
Changed lines of the file:
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@@
 (kicad_sch (version 20211123) (generator eeschema)
   (paper "A4")
+  (junction (at 40.64 134.62) (diameter 0) (color 0 0 0 0)
+  )
   (junction (at 134.62 154.94) (diameter 0) (color 0 0 0 0)
   )
   (junction (at 134.62 87.63) (diameter 0) (color 0 0 0 0)
   )
+  (junction (at 40.64 114.3) (diameter 0) (color 0 0 0 0)
+  )
   (junction (at 167.64 154.94) (diameter 0) (color 0 0 0 0)
   )
@@
   (junction (at 151.13 87.63) (diameter 0) (color 0 0 0 0)
   )
-  (junction (at 83.82 151.13) (diameter 0) (color 0 0 0 0)
-  )
   (junction (at 200.66 154.94) (diameter 0) (color 0 0 0 0)
   )
+  (junction (at 40.64 119.38) (diameter 0) (color 0 0 0 0)
+  )
   (junction (at 101.6 154.94) (diameter 0) (color 0 0 0 0)
   )
+  (junction (at 40.64 104.14) (diameter 0) (color 0 0 0 0)
+  )
+  (junction (at 83.82 142.24) (diameter 0) (color 0 0 0 0)
+  )
   (junction (at 118.11 87.63) (diameter 0) (color 0 0 0 0)
   )
@@
   (junction (at 184.15 154.94) (diameter 0) (color 0 0 0 0)
   )
+  (junction (at 200.66 87.63) (diameter 0) (color 0 0 0 0)
+  )
   (junction (at 86.36 154.94) (diameter 0) (color 0 0 0 0)
   )
-  (junction (at 200.66 87.63) (diameter 0) (color 0 0 0 0)
-  )
   (junction (at 167.64 87.63) (diameter 0) (color 0 0 0 0)
   )
   (junction (at 151.13 154.94) (diameter 0) (color 0 0 0 0)
   )
+  (junction (at 40.64 129.54) (diameter 0) (color 0 0 0 0)
+  )
+  (no_connect (at 55.88 116.84))
+  (no_connect (at 55.88 132.08))
+  (no_connect (at 55.88 101.6))
   (bus_entry (at 180.34 33.02) (size 2.54 -2.54)
     (stroke (width 0) (type default) (color 0 0 0 0))
@@
     (stroke (width 0) (type default) (color 0 0 0 0))
   )
+  (bus (pts (xy 83.82 142.24) (xy 83.82 151.13))
+    (stroke (width 0) (type default) (color 0 0 0 0))
+  )
   (wire (pts (xy 147.32 100.33) (xy 147.32 114.3))
     (stroke (width 0) (type default) (color 0 0 0 0))
@@
     (stroke (width 0) (type default) (color 0 0 0 0))
   )
+  (wire (pts (xy 40.64 134.62) (xy 40.64 139.7))
+    (stroke (width 0) (type default) (color 0 0 0 0))
+  )
   (bus (pts (xy 199.39 97.79) (xy 215.9 97.79))
     (stroke (width 0) (type default) (color 0 0 0 0))
   )
+  (wire (pts (xy 57.15 152.4) (xy 66.04 152.4))
+    (stroke (width 0) (type default) (color 0 0 0 0))
+  )
   (wire (pts (xy 86.36 87.63) (xy 86.36 154.94))
     (stroke (width 0) (type default) (color 0 0 0 0))
@@
     (stroke (width 0) (type default) (color 0 0 0 0))
   )
+  (wire (pts (xy 81.28 154.94) (xy 86.36 154.94))
+    (stroke (width 0) (type default) (color 0 0 0 0))
+  )
   (bus (pts (xy 116.84 97.79) (xy 133.35 97.79))
     (stroke (width 0) (type default) (color 0 0 0 0))
@@
     (stroke (width 0) (type default) (color 0 0 0 0))
   )
+  (wire (pts (xy 40.64 99.06) (xy 40.64 104.14))
+    (stroke (width 0) (type default) (color 0 0 0 0))
+  )
   (bus (pts (xy 128.27 151.13) (xy 144.78 151.13))
     (stroke (width 0) (type default) (color 0 0 0 0))
   )
-  (wire (pts (xy 73.66 154.94) (xy 86.36 154.94))
-    (stroke (width 0) (type default) (color 0 0 0 0))
-  )
   (wire (pts (xy 196.85 33.02) (xy 196.85 46.99))
     (stroke (width 0) (type default) (color 0 0 0 0))
@@
     (stroke (width 0) (type default) (color 0 0 0 0))
   )
+  (bus (pts (xy 73.66 142.24) (xy 83.82 142.24))
+    (stroke (width 0) (type default) (color 0 0 0 0))
+  )
   (wire (pts (xy 130.81 134.62) (xy 130.81 148.59))
     (stroke (width 0) (type default) (color 0 0 0 0))
   )
+  (wire (pts (xy 40.64 119.38) (xy 40.64 129.54))
+    (stroke (width 0) (type default) (color 0 0 0 0))
+  )
+  (wire (pts (xy 40.64 104.14) (xy 40.64 114.3))
+    (stroke (width 0) (type default) (color 0 0 0 0))
+  )
   (bus (pts (xy 166.37 97.79) (xy 182.88 97.79))
     (stroke (width 0) (type default) (color 0 0 0 0))
@@
     (stroke (width 0) (type default) (color 0 0 0 0))
   )
-  (bus (pts (xy 83.82 83.82) (xy 83.82 151.13))
+  (bus (pts (xy 83.82 83.82) (xy 83.82 142.24))
     (stroke (width 0) (type default) (color 0 0 0 0))
   )
@@
     (stroke (width 0) (type default) (color 0 0 0 0))
   )
+  (wire (pts (xy 40.64 114.3) (xy 40.64 119.38))
+    (stroke (width 0) (type default) (color 0 0 0 0))
+  )
   (bus (pts (xy 133.35 97.79) (xy 149.86 97.79))
     (stroke (width 0) (type default) (color 0 0 0 0))
@@
     (stroke (width 0) (type default) (color 0 0 0 0))
   )
+  (wire (pts (xy 40.64 129.54) (xy 40.64 134.62))
+    (stroke (width 0) (type default) (color 0 0 0 0))
+  )
   (wire (pts (xy 130.81 100.33) (xy 130.81 114.3))
     (stroke (width 0) (type default) (color 0 0 0 0))
@@
     (stroke (width 0) (type default) (color 0 0 0 0))
   )
-  (bus (pts (xy 73.66 151.13) (xy 83.82 151.13))
+  (wire (pts (xy 57.15 157.48) (xy 66.04 157.48))
     (stroke (width 0) (type default) (color 0 0 0 0))
   )
   (text "信号補正部\nRegデータバスから送られてくる生のデータ(RAW_DATA)は選択されたレジスタの位置によって反転，非反転が異なる．\n従って選択されたレジスタの物理的な位置を検出し，適切に補正する必要がある．\n\n補正はレジスタ部から送られてくる補正信号を基に反転，非反転を制御し，すべてのビットに対して適切に反転，非反転の処理を加えALUへデータを送る"
-    (at 53.34 177.8 0)
+    (at 55.88 181.61 0)
     (effects (font (size 1.27 1.27)) (justify left bottom))
   )
@@
     (effects (font (size 1.27 1.27)) (justify right bottom))
   )
-  (global_label "RAW_DATA[0..15]" (shape input) (at 73.66 151.13 180) (fields_autoplaced)
+  (global_label "RAW_DATA[0..15]" (shape input) (at 73.66 142.24 180) (fields_autoplaced)
     (effects (font (size 1.27 1.27)) (justify right))
-    (property "Intersheet References" "${INTERSHEET_REFS}" (id 0) (at 55.5231 151.0506 0)
+    (property "Intersheet References" "${INTERSHEET_REFS}" (id 0) (at 55.5231 142.1606 0)
       (effects (font (size 1.27 1.27)) (justify right) hide)
     )
@@
     )
   )
-  (global_label "Correction" (shape input) (at 73.66 154.94 180) (fields_autoplaced)
+  (global_label "Correction" (shape input) (at 57.15 157.48 180) (fields_autoplaced)
     (effects (font (size 1.27 1.27)) (justify right))
-    (property "Intersheet References" "${INTERSHEET_REFS}" (id 0) (at 61.4498 154.8606 0)
+    (property "Intersheet References" "${INTERSHEET_REFS}" (id 0) (at 44.9398 157.4006 0)
       (effects (font (size 1.27 1.27)) (justify right) hide)
     )
   )
+  (symbol (lib_id "power:VCC") (at 57.15 152.4 0) (unit 1)
+    (in_bom yes) (on_board yes) (fields_autoplaced)
+    (property "Reference" "#PWR020" (id 0) (at 57.15 156.21 0)
+      (effects (font (size 1.27 1.27)) hide)
+    )
+    (property "Value" "VCC" (id 1) (at 57.15 148.59 0))
+    (property "Footprint" "" (id 2) (at 57.15 152.4 0)
+      (effects (font (size 1.27 1.27)) hide)
+    )
+    (property "Datasheet" "" (id 3) (at 57.15 152.4 0)
+      (effects (font (size 1.27 1.27)) hide)
+    )
+    (pin "1")
+  )
+  (symbol (lib_id "CD74HCXX:CD74HC00") (at 48.26 116.84 0) (mirror x) (unit 3)
+    (in_bom yes) (on_board yes) (fields_autoplaced)
+    (property "Reference" "U43" (id 0) (at 48.26 107.95 0))
+    (property "Value" "CD74HC00" (id 1) (at 48.26 110.49 0))
+    (property "Footprint" "Package_DIP:DIP-14_W7.62mm" (id 2) (at 43.18 116.84 0)
+      (effects (font (size 1.27 1.27)) hide)
+    )
+    (property "Datasheet" "" (id 3) (at 43.18 116.84 0))
+    (pin "14")
+    (pin "7")
+    (pin "1")
+    (pin "2")
+    (pin "3")
+    (pin "4")
+    (pin "5")
+    (pin "6")
+    (pin "10")
+    (pin "8")
+    (pin "9")
+    (pin "11")
+    (pin "12")
+    (pin "13")
+  )
+  (symbol (lib_id "CD74HCXX:CD74HC00") (at 73.66 154.94 0) (mirror x) (unit 1)
+    (in_bom yes) (on_board yes) (fields_autoplaced)
+    (property "Reference" "U43" (id 0) (at 73.66 146.05 0))
+    (property "Value" "CD74HC00" (id 1) (at 73.66 148.59 0))
+    (property "Footprint" "Package_DIP:DIP-14_W7.62mm" (id 2) (at 68.58 154.94 0)
+      (effects (font (size 1.27 1.27)) hide)
+    )
+    (property "Datasheet" "" (id 3) (at 68.58 154.94 0))
+    (pin "14")
+    (pin "7")
+    (pin "1")
+    (pin "2")
+    (pin "3")
+    (pin "4")
+    (pin "5")
+    (pin "6")
+    (pin "10")
+    (pin "8")
+    (pin "9")
+    (pin "11")
+    (pin "12")
+    (pin "13")
+  )
+  (symbol (lib_id "CD74HCXX:CD74HC00") (at 48.26 101.6 0) (mirror x) (unit 2)
+    (in_bom yes) (on_board yes) (fields_autoplaced)
+    (property "Reference" "U43" (id 0) (at 48.26 92.71 0))
+    (property "Value" "CD74HC00" (id 1) (at 48.26 95.25 0))
+    (property "Footprint" "Package_DIP:DIP-14_W7.62mm" (id 2) (at 43.18 101.6 0)
+      (effects (font (size 1.27 1.27)) hide)
+    )
+    (property "Datasheet" "" (id 3) (at 43.18 101.6 0))
+    (pin "14")
+    (pin "7")
+    (pin "1")
+    (pin "2")
+    (pin "3")
+    (pin "4")
+    (pin "5")
+    (pin "6")
+    (pin "10")
+    (pin "8")
+    (pin "9")
+    (pin "11")
+    (pin "12")
+    (pin "13")
+  )
+  (symbol (lib_id "power:GND") (at 40.64 139.7 0) (unit 1)
+    (in_bom yes) (on_board yes) (fields_autoplaced)
+    (property "Reference" "#PWR019" (id 0) (at 40.64 146.05 0)
+      (effects (font (size 1.27 1.27)) hide)
+    )
+    (property "Value" "GND" (id 1) (at 40.64 144.78 0))
+    (property "Footprint" "" (id 2) (at 40.64 139.7 0)
+      (effects (font (size 1.27 1.27)) hide)
+    )
+    (property "Datasheet" "" (id 3) (at 40.64 139.7 0)
+      (effects (font (size 1.27 1.27)) hide)
+    )
+    (pin "1")
+  )
+  (symbol (lib_id "CD74HCXX:CD74HC00") (at 48.26 132.08 0) (mirror x) (unit 4)
+    (in_bom yes) (on_board yes) (fields_autoplaced)
+    (property "Reference" "U43" (id 0) (at 48.26 123.19 0))
+    (property "Value" "CD74HC00" (id 1) (at 48.26 125.73 0))
+    (property "Footprint" "Package_DIP:DIP-14_W7.62mm" (id 2) (at 43.18 132.08 0)
+      (effects (font (size 1.27 1.27)) hide)
+    )
+    (property "Datasheet" "" (id 3) (at 43.18 132.08 0))
+    (pin "14")
+    (pin "7")
+    (pin "1")
+    (pin "2")
+    (pin "3")
+    (pin "4")
+    (pin "5")
+    (pin "6")
+    (pin "10")
+    (pin "8")
+    (pin "9")
+    (pin "11")
+    (pin "12")
+    (pin "13")
+  )
   (sheet (at 208.28 114.3) (size 12.7 20.32)
