File: nlp-16a/Hardware/A_B_BUS_Ctrl/A_B_BUS_Ctrl/Correction.kicad_sch (KiCad schematic)
At the start: 4 parts

Commit message: 配線作業開始
Parts:
- U16: renamed from U?; footprint (none) -> Package_DIP:DIP-14_W7.62mm
Changed lines of the file:
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@@
   (symbol (lib_id "CD74HCXX:CD74HC00") (at 168.91 90.17 0) (mirror x) (unit 3)
     (in_bom yes) (on_board yes) (fields_autoplaced)
-    (property "Reference" "U?" (id 0) (at 168.91 81.28 0))
+    (property "Reference" "U16" (id 0) (at 168.91 81.28 0))
     (property "Value" "CD74HC00" (id 1) (at 168.91 83.82 0))
-    (property "Footprint" "" (id 2) (at 163.83 90.17 0))
+    (property "Footprint" "Package_DIP:DIP-14_W7.62mm" (id 2) (at 163.83 90.17 0)
+      (effects (font (size 1.27 1.27)) hide)
+    )
     (property "Datasheet" "" (id 3) (at 163.83 90.17 0))
     (pin "14")
@@
   (symbol (lib_id "CD74HCXX:CD74HC00") (at 148.59 96.52 0) (unit 2)
     (in_bom yes) (on_board yes) (fields_autoplaced)
-    (property "Reference" "U?" (id 0) (at 148.59 87.63 0))
+    (property "Reference" "U16" (id 0) (at 148.59 87.63 0))
     (property "Value" "CD74HC00" (id 1) (at 148.59 90.17 0))
-    (property "Footprint" "" (id 2) (at 143.51 96.52 0))
+    (property "Footprint" "Package_DIP:DIP-14_W7.62mm" (id 2) (at 143.51 96.52 0)
+      (effects (font (size 1.27 1.27)) hide)
+    )
     (property "Datasheet" "" (id 3) (at 143.51 96.52 0))
     (pin "14")
@@
   (symbol (lib_id "CD74HCXX:CD74HC00") (at 127 90.17 0) (mirror x) (unit 1)
     (in_bom yes) (on_board yes) (fields_autoplaced)
-    (property "Reference" "U?" (id 0) (at 127 81.28 0))
+    (property "Reference" "U16" (id 0) (at 127 81.28 0))
     (property "Value" "CD74HC00" (id 1) (at 127 83.82 0))
-    (property "Footprint" "" (id 2) (at 121.92 90.17 0))
+    (property "Footprint" "Package_DIP:DIP-14_W7.62mm" (id 2) (at 121.92 90.17 0)
+      (effects (font (size 1.27 1.27)) hide)
+    )
     (property "Datasheet" "" (id 3) (at 121.92 90.17 0))
     (pin "14")
@@
   (symbol (lib_id "CD74HCXX:CD74HC00") (at 148.59 83.82 0) (mirror x) (unit 4)
     (in_bom yes) (on_board yes) (fields_autoplaced)
-    (property "Reference" "U?" (id 0) (at 148.59 74.93 0))
+    (property "Reference" "U16" (id 0) (at 148.59 74.93 0))
     (property "Value" "CD74HC00" (id 1) (at 148.59 77.47 0))
-    (property "Footprint" "" (id 2) (at 143.51 83.82 0))
+    (property "Footprint" "Package_DIP:DIP-14_W7.62mm" (id 2) (at 143.51 83.82 0)
+      (effects (font (size 1.27 1.27)) hide)
+    )
     (property "Datasheet" "" (id 3) (at 143.51 83.82 0))
     (pin "14")
