File: nlp-16a/Hardware/Y_BUS_Ctrl/TMP_Reg.kicad_sch (KiCad schematic)
At the start: 32 parts

Commit message: Yバスだいたい配線完了
Changed lines of the file:
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@@
     (effects (font (size 1.27 1.27)) (justify left bottom))
   )
-  (global_label "IN" (shape input) (at 60.96 143.51 180) (fields_autoplaced)
+  (global_label "IN[0..15]" (shape input) (at 60.96 143.51 180) (fields_autoplaced)
     (effects (font (size 1.27 1.27)) (justify right))
-    (property "Intersheet References" "${INTERSHEET_REFS}" (id 0) (at 56.6117 143.4306 0)
+    (property "Intersheet References" "${INTERSHEET_REFS}" (id 0) (at 50.0802 143.4306 0)
       (effects (font (size 1.27 1.27)) (justify right) hide)
     )
   )
-  (global_label "OUT" (shape output) (at 231.14 36.83 0) (fields_autoplaced)
+  (global_label "OUT[0..15]" (shape output) (at 231.14 36.83 0) (fields_autoplaced)
     (effects (font (size 1.27 1.27)) (justify left))
-    (property "Intersheet References" "${INTERSHEET_REFS}" (id 0) (at 237.1817 36.7506 0)
+    (property "Intersheet References" "${INTERSHEET_REFS}" (id 0) (at 243.7131 36.7506 0)
       (effects (font (size 1.27 1.27)) (justify left) hide)
     )

Commit message: YバスTMPRegリファレンス割り当て
Parts:
- added R? (x16): R, symbol Device:R
Connections:
- net OUT0: now also R?.2; no longer D?.2 (A)
- net OUT1: now also R?.2; no longer D?.2 (A)
- net OUT10: now also R?.2; no longer D?.2 (A)
- net OUT11: now also R?.2; no longer D?.2 (A)
- net OUT12: now also R?.2; no longer D?.2 (A)
- net OUT13: now also R?.2; no longer D?.2 (A)
- net OUT14: now also R?.2; no longer D?.2 (A)
- net OUT15: now also R?.2; no longer D?.2 (A)
- net OUT2: now also R?.2; no longer D?.2 (A)
- net OUT3: now also R?.2; no longer D?.2 (A)
- net OUT4: now also R?.2; no longer D?.2 (A)
- net OUT5: now also R?.2; no longer D?.2 (A)
- net OUT6: now also R?.2; no longer D?.2 (A)
- net OUT7: now also R?.2; no longer D?.2 (A)
- net OUT8: now also R?.2; no longer D?.2 (A)
- net OUT9: now also R?.2; no longer D?.2 (A)
- new net Reg0/Q: D?.2 (A), R?.1
- new net Reg1/Q: D?.2 (A), R?.1
- new net Reg10/Q: D?.2 (A), R?.1
- new net Reg11/Q: D?.2 (A), R?.1
- new net Reg12/Q: D?.2 (A), R?.1
- new net Reg13/Q: D?.2 (A), R?.1
- new net Reg14/Q: D?.2 (A), R?.1
- new net Reg15/Q: D?.2 (A), R?.1
- new net Reg2/Q: D?.2 (A), R?.1
- new net Reg3/Q: D?.2 (A), R?.1
- new net Reg4/Q: D?.2 (A), R?.1
- new net Reg5/Q: D?.2 (A), R?.1
- new net Reg6/Q: D?.2 (A), R?.1
- new net Reg7/Q: D?.2 (A), R?.1
- new net Reg8/Q: D?.2 (A), R?.1
- new net Reg9/Q: D?.2 (A), R?.1

Commit message: Yバス制御 配置の決定，リファレンスの割り当て，ERCの確認完了
Parts:
- gave numbers to parts that had none: 34

Commit message: Y BUS制御の基板をとりあえず描いた．ビアとかはまた後で
Parts:
- removed R1, R10, R11, R12, R13, R14, R15, R16, R2, R3, R4, R5, R6, R7, R8, R9: R, symbol Device:R
- D1, D10, D11, D12, D13, D14, D15, D16, D2, D3, D4, D5, D6, D7, D8, D9: footprint (none) -> LED_THT:LED_D3.0mm
Connections:
- net Reg0/Q is gone; now on net OUT0: D1.2 (A)
- net Reg1/Q is gone; now on net OUT1: D2.2 (A)
- net Reg10/Q is gone; now on net OUT10: D11.2 (A)
- net Reg11/Q is gone; now on net OUT11: D12.2 (A)
- net Reg12/Q is gone; now on net OUT12: D13.2 (A)
- net Reg13/Q is gone; now on net OUT13: D14.2 (A)
- net Reg14/Q is gone; now on net OUT14: D15.2 (A)
- net Reg15/Q is gone; now on net OUT15: D16.2 (A)
- net Reg2/Q is gone; now on net OUT2: D3.2 (A)
- net Reg3/Q is gone; now on net OUT3: D4.2 (A)
- net Reg4/Q is gone; now on net OUT4: D5.2 (A)
- net Reg5/Q is gone; now on net OUT5: D6.2 (A)
- net Reg6/Q is gone; now on net OUT6: D7.2 (A)
- net Reg7/Q is gone; now on net OUT7: D8.2 (A)
- net Reg8/Q is gone; now on net OUT8: D9.2 (A)
- net Reg9/Q is gone; now on net OUT9: D10.2 (A)
