File: nlp-16a/Hardware/Y_BUS_Ctrl/Y_BUS_Ctrl.kicad_pcb (KiCad board)
At the start: 2 copper layers, 209.6 x 154.9 mm, 141 parts, among them J1 Conn_02x20_Odd_Even, J2 Conn_02x20_Odd_Even, J3 Conn_02x10_Odd_Even, J4 Conn_02x10_Counter_Clockwise, J5 Screw_Terminal_01x02, U1 CD74HC00, U10 CD74HC00, U11 CD74HC00, U12 CD74HC00, U13 CD74HC00, U14 CD74HC00, U15 CD74HC00, U16 CD74HC00, U17 CD74HC00, U18 CD74HC00, U19 CD74HC00, U2 CD74HC00, U20 CD74HC00, U21 CD74HC00, U22 CD74HC00, U23 CD74HC00, U24 CD74HC00, U25 CD74HC00, U26 CD74HC00, U27 CD74HC00, U28 CD74HC00, U29 CD74HC00, U3 CD74HC00, U30 CD74HC00, U31 CD74HC00, U32 CD74HC00, U33 CD74HC00, U34 CD74HC00, U35 CD74HC00, U36 CD74HC00, U37 CD74HC00, U38 CD74HC00, U39 CD74HC00, U4 CD74HC00, U40 CD74HC00, U41 CD74HC00, U42 CD74HC00, U5 CD74HC00, U6 CD74HC00, U7 CD74HC00, U8 CD74HC00, U9 CD74HC00

Commit message: Y-BUS制御完成
Parts:
- added R33: 22, Resistor_SMD:R_0603_1608Metric_Pad0.98x0.95mm_HandSolder, F.Cu at (109.9, 43.2)
- added U43: CD74HC00, Package_DIP:DIP-14_W7.62mm, F.Cu at (145.4, 109.2)
- moved G*** 202.2 mm to (226.7, 40.6), turned to 0 degrees
Connections:
- J1 pad 36: phi1 -> phi1_bus
- U1 pad 2: phi1 -> phi1_Reg2
- U1 pad 5: phi1 -> phi1_Reg2
- U10 pad 2: phi1 -> phi1_Reg1
- U10 pad 5: phi1 -> phi1_Reg1
- U11 pad 2: phi1 -> phi1_Reg1
- U11 pad 5: phi1 -> phi1_Reg1
- U12 pad 2: phi1 -> phi1_Reg1
- U12 pad 5: phi1 -> phi1_Reg1
- U13 pad 2: phi1 -> phi1_Reg1
- U13 pad 5: phi1 -> phi1_Reg1
- U14 pad 2: phi1 -> phi1_Reg1
- U14 pad 5: phi1 -> phi1_Reg1
- U15 pad 2: phi1 -> phi1_Reg1
- U15 pad 5: phi1 -> phi1_Reg1
- U16 pad 2: phi1 -> phi1_Reg1
- U16 pad 5: phi1 -> phi1_Reg1
- U2 pad 2: phi1 -> phi1_Reg2
- U2 pad 5: phi1 -> phi1_Reg2
- U3 pad 2: phi1 -> phi1_Reg2
- U3 pad 5: phi1 -> phi1_Reg2
- U4 pad 2: phi1 -> phi1_Reg2
- U4 pad 5: phi1 -> phi1_Reg2
- U5 pad 2: phi1 -> phi1_Reg2
- U5 pad 5: phi1 -> phi1_Reg2
- U6 pad 2: phi1 -> phi1_Reg2
- U6 pad 5: phi1 -> phi1_Reg2
- U7 pad 2: phi1 -> phi1_Reg2
- U7 pad 5: phi1 -> phi1_Reg2
- U8 pad 2: phi1 -> phi1_Reg2
- U8 pad 5: phi1 -> phi1_Reg2
- U9 pad 2: phi1 -> phi1_Reg1
- U9 pad 5: phi1 -> phi1_Reg1
Routing:
- net phi1: track 652.1 -> 111.7 mm, vias 32 -> 2
- net Net-(R33-Pad1): track 0.00 -> 264.0 mm, vias 0 -> 3
- net phi1_Reg2: track 0.00 -> 236.6 mm, vias 0 -> 17
- net phi1_Reg1: track 0.00 -> 221.9 mm, vias 0 -> 16
- net Net-(U43-Pad10): track 0.00 -> 25.4 mm
- net phi1_bus: track 0.00 -> 14.5 mm
- net VCC: track 1337.8 -> 1339.9 mm
- net phi2: track 230.2 -> 229.2 mm
- net GND: vias 0 -> 453
Other:
- board text added: "MEM RegF RegE RegD"
- board text removed: "MEM RedF RegE RegD"
