File: nlp-16a/Hardware/A_BUS_Ctrl/address_decoder.kicad_sch (KiCad schematic)
At the start: 21 parts, among them U41 CD74HC00, U42 CD74HC00, U43 CD74HC00

Commit message: テストで見つかった不具合を修正(れジスタアドレスデコーダ，Addrの内部処理の方法を変更)
Changed lines of the file:
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@@
   (junction (at 119.38 149.86) (diameter 0) (color 0 0 0 0)
   )
-  (junction (at 195.58 140.97) (diameter 0) (color 0 0 0 0)
-  )
   (junction (at 60.96 66.04) (diameter 0) (color 0 0 0 0)
   )
@@
     (stroke (width 0) (type default) (color 0 0 0 0))
   )
-  (wire (pts (xy 191.77 139.7) (xy 191.77 140.97))
-    (stroke (width 0) (type default) (color 0 0 0 0))
-  )
   (wire (pts (xy 165.1 149.86) (xy 274.32 149.86))
     (stroke (width 0) (type default) (color 0 0 0 0))
@@
     (stroke (width 0) (type default) (color 0 0 0 0))
   )
+  (wire (pts (xy 191.77 139.7) (xy 191.77 161.29))
+    (stroke (width 0) (type default) (color 0 0 0 0))
+  )
   (bus (pts (xy 140.97 41.91) (xy 163.83 41.91))
     (stroke (width 0) (type default) (color 0 0 0 0))
@@
     (stroke (width 0) (type default) (color 0 0 0 0))
   )
+  (wire (pts (xy 60.96 22.86) (xy 60.96 20.32))
+    (stroke (width 0) (type default) (color 0 0 0 0))
+  )
+  (wire (pts (xy 256.54 81.28) (xy 274.32 81.28))
+    (stroke (width 0) (type default) (color 0 0 0 0))
+  )
+  (wire (pts (xy 82.55 52.07) (xy 82.55 88.9))
+    (stroke (width 0) (type default) (color 0 0 0 0))
+  )
+  (wire (pts (xy 138.43 114.3) (xy 138.43 128.27))
+    (stroke (width 0) (type default) (color 0 0 0 0))
+  )
+  (wire (pts (xy 15.24 46.99) (xy 21.59 46.99))
+    (stroke (width 0) (type default) (color 0 0 0 0))
+  )
+  (wire (pts (xy 60.96 68.58) (xy 60.96 66.04))
+    (stroke (width 0) (type default) (color 0 0 0 0))
+  )
+  (wire (pts (xy 241.3 73.66) (xy 241.3 93.98))
+    (stroke (width 0) (type default) (color 0 0 0 0))
+  )
   (wire (pts (xy 252.73 114.3) (xy 252.73 128.27))
     (stroke (width 0) (type default) (color 0 0 0 0))
   )
-  (wire (pts (xy 60.96 22.86) (xy 60.96 20.32))
-    (stroke (width 0) (type default) (color 0 0 0 0))
-  )
-  (wire (pts (xy 256.54 81.28) (xy 274.32 81.28))
-    (stroke (width 0) (type default) (color 0 0 0 0))
-  )
-  (wire (pts (xy 82.55 52.07) (xy 82.55 88.9))
-    (stroke (width 0) (type default) (color 0 0 0 0))
-  )
-  (wire (pts (xy 138.43 114.3) (xy 138.43 128.27))
-    (stroke (width 0) (type default) (color 0 0 0 0))
-  )
-  (wire (pts (xy 15.24 46.99) (xy 21.59 46.99))
-    (stroke (width 0) (type default) (color 0 0 0 0))
-  )
-  (wire (pts (xy 60.96 68.58) (xy 60.96 66.04))
-    (stroke (width 0) (type default) (color 0 0 0 0))
-  )
-  (wire (pts (xy 241.3 73.66) (xy 241.3 93.98))
-    (stroke (width 0) (type default) (color 0 0 0 0))
-  )
   (wire (pts (xy 58.42 91.44) (xy 127 91.44))
     (stroke (width 0) (type default) (color 0 0 0 0))
@@
     (stroke (width 0) (type default) (color 0 0 0 0))
   )
-  (wire (pts (xy 191.77 140.97) (xy 195.58 140.97))
-    (stroke (width 0) (type default) (color 0 0 0 0))
-  )
   (wire (pts (xy 82.55 88.9) (xy 82.55 154.94))
     (stroke (width 0) (type default) (color 0 0 0 0))
@@
   )
   (wire (pts (xy 58.42 66.04) (xy 58.42 91.44))
+    (stroke (width 0) (type default) (color 0 0 0 0))
+  )
+  (wire (pts (xy 190.5 161.29) (xy 191.77 161.29))
     (stroke (width 0) (type default) (color 0 0 0 0))
   )
@@
       (effects (font (size 1.27 1.27)) (justify right) hide)
     )
+  )
+  (global_label "~INTERNAL" (shape input) (at 190.5 161.29 180) (fields_autoplaced)
+    (effects (font (size 1.27 1.27)) (justify right))
+    (property "Intersheet References" "${INTERSHEET_REFS}" (id 0) (at 178.4107 161.2106 0)
+      (effects (font (size 1.27 1.27)) (justify right) hide)
+    )

Commit message: A BUS制御 IVとIR3のアドレスの処理変更を反映
Changed lines of the file:
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@@
     )
   )
-  (global_label "~IV" (shape input) (at 175.26 97.79 180) (fields_autoplaced)
+  (global_label "~IV" (shape input) (at 152.4 97.79 180) (fields_autoplaced)
     (effects (font (size 1.27 1.27)) (justify right))
-    (property "Intersheet References" "${INTERSHEET_REFS}" (id 0) (at 170.2464 97.7106 0)
+    (property "Intersheet References" "${INTERSHEET_REFS}" (id 0) (at 147.3864 97.7106 0)
       (effects (font (size 1.27 1.27)) (justify right) hide)
     )
@@
     )
   )
-  (global_label "~IR3" (shape input) (at 152.4 97.79 180) (fields_autoplaced)
+  (global_label "~IR3" (shape input) (at 175.26 97.79 180) (fields_autoplaced)
     (effects (font (size 1.27 1.27)) (justify right))
-    (property "Intersheet References" "${INTERSHEET_REFS}" (id 0) (at 145.9955 97.7106 0)
+    (property "Intersheet References" "${INTERSHEET_REFS}" (id 0) (at 168.8555 97.7106 0)
       (effects (font (size 1.27 1.27)) (justify right) hide)
     )
