File: nlp-16a/Hardware/Instruction_decoder/Instruction_decoder.kicad_pcb (KiCad board)
At the start: 2 copper layers, 209.6 x 154.9 mm, 119 parts, among them J1 Conn_02x10_Odd_Even, J2 Conn_02x10_Odd_Even, J3 Screw_Terminal_01x02, J4 Conn_02x10_Counter_Clockwise, J5 Conn_02x10_Counter_Clockwise, U1 State_hold_unit, U10 State_hold_unit, U11 State_hold_unit, U12 State_hold_unit, U13 State_hold_unit, U14 State_hold_unit, U15 State_hold_unit, U16 State_hold_unit, U17 State_hold_unit, U18 State_hold_unit, U19 State_hold_unit, U2 State_hold_unit, U20 State_hold_unit, U21 State_hold_unit, U22 State_hold_unit, U23 State_hold_unit, U24 State_hold_unit, U25 State_hold_unit, U26 State_hold_unit, U27 State_hold_unit, U28 State_hold_unit, U29 State_hold_unit, U3 State_hold_unit, U30 State_hold_unit, U31 State_hold_unit, U32 State_hold_unit, U33 State_hold_unit, U34 State_hold_unit, U35 State_hold_unit, U36 State_hold_unit, U37 State_hold_unit, U38 State_hold_unit, U39 State_hold_unit, U4 State_hold_unit, U40 State_hold_unit, U41 State_hold_unit, U42 State_hold_unit, U43 State_hold_unit, U44 State_hold_unit, U45 State_hold_unit, U46 State_hold_unit, U47 State_hold_unit, U48 State_hold_unit, U49 CD74HC00, U5 State_hold_unit, U50 CD74HC00, U51 CD74HC00, U52 CD74HC00, U53 CD74HC00, U54 CD74HC00, U55 CD74HC00, U56 CD74HC00, U57 CD74HC00, U58 CD74HC00, U59 CD74HC00, U6 State_hold_unit, U60 CD74HC00, U61 CD74HC00, U62 CD74HC00, U63 CD74HC00, U64 CD74HC00, U65 CD74HC00, U66 CD74HC00, U67 CD74HC00, U68 CD74HC00, U69 CD74HC00, U7 State_hold_unit, U70 CD74HC00, U71 CD74HC00, U72 CD74HC00, U73 CD74HC00, U74 CD74HC00, U75 CD74HC00, U76 CD74HC00, U77 CD74HC00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

Commit message: 基板設計 進捗
Parts:
- moved C7 158.8 mm to (40.6, 54.0), turned to 180 degrees
- moved C22 51.0 mm to (111.8, 220.6)
- moved C23 51.0 mm to (111.8, 212.5)
- moved C6 50.6 mm to (93.7, 216.5)
- moved C17 50.6 mm to (102.7, 216.5)
- moved C13 50.4 mm to (102.7, 212.5)
- moved C16 47.4 mm to (84.6, 228.7)
- moved C8 47.1 mm to (93.7, 232.7)
- moved C15 46.0 mm to (102.7, 228.7)
- moved C9 45.0 mm to (120.8, 212.5)
- moved C20 44.2 mm to (84.6, 216.5)
- moved C12 43.4 mm to (93.7, 224.6)
- moved C19 42.2 mm to (84.6, 232.7)
- moved C10 41.2 mm to (93.7, 220.6)
- moved C11 40.6 mm to (93.7, 228.7)
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Connections:
- J2 pad 12: 3word -> ~{Seed_pluse}
- J2 pad 8: ~{Seed_pluse} -> 3word
- J4 pad 11: unconnected-(J4-Pad11) -> ~{IR3_Y}
- J4 pad 13: ~{IR3_Y} -> Acc_Y
- U16 pad 5: ~{Acc_Y} -> ~{AccWR}
- U22 pad 3: WB -> ~{INTERNAL_Y}
- U22 pad 4: WB -> ~{INTERNAL_Y}
- U22 pad 5: unconnected-(U22-Pad5) -> ~{WB}
- U49 pad 1: Net-(U49-Pad1) -> OP7
- U49 pad 4: OP7 -> Net-(U49-Pad3)
- U49 pad 6: Net-(U49-Pad1) -> Net-(U54-Pad4)
- U50 pad 4: Net-(U49-Pad1) -> Net-(U49-Pad3)
- U50 pad 5: Net-(U49-Pad1) -> Net-(U49-Pad3)
- U54 pad 4: Net-(U49-Pad3) -> Net-(U54-Pad4)
- U56 pad 2: ~{Acc_Y} -> ~{AccWR}
- U59 pad 13: WB -> ~{INTERNAL_Y}
- U59 pad 9: WB -> ~{INTERNAL_Y}
- U63 pad 4: Net-(U36-Pad5) -> Net-(U63-Pad3)
- U63 pad 5: Net-(U63-Pad3) -> Net-(U36-Pad5)
- U70 pad 4: ~{OP->} -> ~{AccWR}
- U70 pad 5: ~{RA3} -> ~{WB}
- U70 pad 6: ~{INTERNAL_Y} -> Acc_Y
- U80 pad 12: Net-(U75-Pad8) -> Net-(U80-Pad12)
- U80 pad 13: Net-(U80-Pad13) -> Net-(U75-Pad8)
- U80 pad 3: Net-(U80-Pad13) -> Net-(U80-Pad12)
Routing:
- net VCC: track 0.00 -> 1162.7 mm
- net GND: track 59.3 -> 1195.5 mm, vias 0 -> 14
- net ~{RAM_STORE->}: track 0.00 -> 391.0 mm, vias 0 -> 4
- net 3word: track 0.00 -> 234.6 mm, vias 0 -> 2
- net ~{SP_INC_POP->}: track 12.0 -> 237.1 mm, vias 0 -> 2
- net END_EXE: track 0.00 -> 220.9 mm, vias 0 -> 2
- net ~{PUSH_EXE}: track 2.54 -> 216.3 mm, vias 0 -> 2
- net OP6: track 7.32 -> 184.7 mm, vias 0 -> 5
- net OP1: track 144.7 -> 321.0 mm, vias 0 -> 4
- net ~{->SP_INC_POP}: track 42.5 -> 216.0 mm, vias 1 -> 4
- net Y_Flag_sel: track 16.5 -> 169.7 mm, vias 0 -> 2
- net OP5: track 246.2 -> 397.6 mm, vias 3 -> 10
- net Net-(U78-Pad10): track 8.68 -> 155.8 mm, vias 0 -> 2
- net ~{Fetch_END2}: track 0.00 -> 146.8 mm, vias 0 -> 2
- net ~{INC_ALU}: track 0.00 -> 141.3 mm, vias 0 -> 2
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- added copper zone on B.Cu, net GND
- added copper zone on F.Cu, net GND
