File: nlp-16a/Hardware/Instruction_decoder/Interrupt.kicad_sch (KiCad schematic)
At the start: 18 parts

Commit message: 命令デコーダ ロジック部の設計だいたい完了git statusgit statusやったぜ
Parts:
- removed U? (x3): CD74HC00, Package_DIP:DIP-14_W7.62mm, symbol CD74HCXX:CD74HC00
Connections:
- net ~{IV_JMP->}: now reaches U?.5 (~{Q})
- net ~{->IV_JMP}: now reaches U?.5 (~{Q})
- net ~{IP_SAVE->}: now reaches U?.5 (~{Q})
- net ~{Flag_SAVE->}: now reaches U?.5 (~{Q})
- net ~{->RAM1} renamed ~{->IP_SAVE}
- net ~{->RAM2} renamed ~{->Flag_SAVE}
- net ~{->SP1} renamed ~{->SP_DEC_INT1}
- net ~{->SP2} renamed ~{->SP_DEC_INT2}
- net ~{SP->/DEC1} renamed ~{SP_DEC_INT1->}
- net ~{SP->/DEC2} renamed ~{SP_DEC_INT2->}
- no-connect marks 12 -> 14
Other:
- note removed: "->RAM"
- note removed: "->SP"
- note removed: "SP/DEC"
- moved on the sheet: U?

Commit message: アノテーションまで完了．基板設計に入る
Parts:
- removed U? (x2): State_hold_unit, symbol State_hold_unit:State_hold_unit
- added unit 1 of U62
- gave numbers to parts that had none: 11
Connections:
- net GND: now also U62.7 (GND)
- net INT: now also U62.1
- net VCC: now also U62.14 (VCC)
- net ~{FETCH_INT}: now also U62.10, U62.11; no longer U62.3
- net ~{INT_FETCH}: now also U62.4; no longer U62.1
- net at U39.1 (D): now also U62.6; no longer U62.3
- net ~{->IV_JMP} renamed ~{->IV_JMP/END_INT}
- new net: U62.13, U62.3
- new net: U62.5, U62.8
- new net INT_EN: U62.2
- new net INT_START: U62.12, U62.9
- no-connect marks 14 -> 10
Other:
- note added: "Hで割り込み開始"
- note added: "ソフト割込み"
- moved on the sheet: U62B, U62C, U62D

Commit message: 基板設計 今日はとりあえずここまで
Parts:
- U39, U40, U41, U42, U43, U44, U45, U46, U47, U48: footprint (none) -> Connector_PinSocket_2.54mm:PinSocket_1x05_P2.54mm_Vertical
Changed lines of the file:
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@@
     (property "Reference" "U47" (id 0) (at 149.86 132.08 0))
     (property "Value" "State_hold_unit" (id 1) (at 149.86 134.62 0))
-    (property "Footprint" "" (id 2) (at 149.86 135.89 0)
+    (property "Footprint" "Connector_PinSocket_2.54mm:PinSocket_1x05_P2.54mm_Vertical" (id 2) (at 149.86 135.89 0)
       (effects (font (size 1.27 1.27)) hide)
     )
@@
     (property "Reference" "U46" (id 0) (at 181.61 106.68 0))
     (property "Value" "State_hold_unit" (id 1) (at 181.61 109.22 0))
-    (property "Footprint" "" (id 2) (at 181.61 110.49 0)
+    (property "Footprint" "Connector_PinSocket_2.54mm:PinSocket_1x05_P2.54mm_Vertical" (id 2) (at 181.61 110.49 0)
       (effects (font (size 1.27 1.27)) hide)
     )
@@
     (property "Reference" "U43" (id 0) (at 86.36 106.68 0))
     (property "Value" "State_hold_unit" (id 1) (at 86.36 109.22 0))
-    (property "Footprint" "" (id 2) (at 86.36 110.49 0)
+    (property "Footprint" "Connector_PinSocket_2.54mm:PinSocket_1x05_P2.54mm_Vertical" (id 2) (at 86.36 110.49 0)
       (effects (font (size 1.27 1.27)) hide)
     )
@@
     (property "Reference" "U42" (id 0) (at 181.61 81.28 0))
     (property "Value" "State_hold_unit" (id 1) (at 181.61 83.82 0))
-    (property "Footprint" "" (id 2) (at 181.61 85.09 0)
+    (property "Footprint" "Connector_PinSocket_2.54mm:PinSocket_1x05_P2.54mm_Vertical" (id 2) (at 181.61 85.09 0)
       (effects (font (size 1.27 1.27)) hide)
     )
@@
     (property "Reference" "U40" (id 0) (at 118.11 81.28 0))
     (property "Value" "State_hold_unit" (id 1) (at 118.11 83.82 0))
-    (property "Footprint" "" (id 2) (at 118.11 85.09 0)
+    (property "Footprint" "Connector_PinSocket_2.54mm:PinSocket_1x05_P2.54mm_Vertical" (id 2) (at 118.11 85.09 0)
       (effects (font (size 1.27 1.27)) hide)
     )
@@
     (property "Reference" "U48" (id 0) (at 181.61 132.08 0))
     (property "Value" "State_hold_unit" (id 1) (at 181.61 134.62 0))
-    (property "Footprint" "" (id 2) (at 181.61 135.89 0)
+    (property "Footprint" "Connector_PinSocket_2.54mm:PinSocket_1x05_P2.54mm_Vertical" (id 2) (at 181.61 135.89 0)
       (effects (font (size 1.27 1.27)) hide)
     )
@@
     (property "Reference" "U39" (id 0) (at 86.36 81.28 0))
     (property "Value" "State_hold_unit" (id 1) (at 86.36 83.82 0))
-    (property "Footprint" "" (id 2) (at 86.36 85.09 0)
+    (property "Footprint" "Connector_PinSocket_2.54mm:PinSocket_1x05_P2.54mm_Vertical" (id 2) (at 86.36 85.09 0)
       (effects (font (size 1.27 1.27)) hide)
     )
@@
     (property "Reference" "U41" (id 0) (at 149.86 81.28 0))
     (property "Value" "State_hold_unit" (id 1) (at 149.86 83.82 0))
-    (property "Footprint" "" (id 2) (at 149.86 85.09 0)
+    (property "Footprint" "Connector_PinSocket_2.54mm:PinSocket_1x05_P2.54mm_Vertical" (id 2) (at 149.86 85.09 0)
       (effects (font (size 1.27 1.27)) hide)
     )
@@
     (property "Reference" "U44" (id 0) (at 118.11 106.68 0))
     (property "Value" "State_hold_unit" (id 1) (at 118.11 109.22 0))
-    (property "Footprint" "" (id 2) (at 118.11 110.49 0)
+    (property "Footprint" "Connector_PinSocket_2.54mm:PinSocket_1x05_P2.54mm_Vertical" (id 2) (at 118.11 110.49 0)
       (effects (font (size 1.27 1.27)) hide)
     )
@@
     (property "Reference" "U45" (id 0) (at 149.86 106.68 0))
     (property "Value" "State_hold_unit" (id 1) (at 149.86 109.22 0))
-    (property "Footprint" "" (id 2) (at 149.86 110.49 0)
-      (effects (font (size 1.27 1.27)) hide)
-    )
+    (property "Footprint" "Connector_PinSocket_2.54mm:PinSocket_1x05_P2.54mm_Vertical" (id 2) (at 149.86 110.49 0)
+      (effects (font (size 1.27 1.27)) hide)
+    )

Commit message: 命令デコーダ完了！！
Connections:
- net phi2_2: now reaches U43.2 (G)
- net phi1_2: now reaches U44.2 (G)
- no-connect marks 10 -> 8
Changed lines of the file:
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@@
   (no_connect (at 171.45 144.78))
   (no_connect (at 171.45 93.98))
-  (no_connect (at 107.95 119.38))
-  (no_connect (at 76.2 119.38))
   (no_connect (at 139.7 93.98))
   (no_connect (at 139.7 119.38))
@@
     (stroke (width 0) (type default) (color 0 0 0 0))
   )
+  (wire (pts (xy 105.41 124.46) (xy 105.41 119.38))
+    (stroke (width 0) (type default) (color 0 0 0 0))
+  )
   (wire (pts (xy 172.72 66.04) (xy 172.72 58.42))
     (stroke (width 0) (type default) (color 0 0 0 0))
@@
     (stroke (width 0) (type default) (color 0 0 0 0))
   )
+  (wire (pts (xy 105.41 119.38) (xy 107.95 119.38))
+    (stroke (width 0) (type default) (color 0 0 0 0))
+  )
   (wire (pts (xy 200.66 104.14) (xy 97.79 104.14))
     (stroke (width 0) (type default) (color 0 0 0 0))
@@
     (stroke (width 0) (type default) (color 0 0 0 0))
   )
+  (wire (pts (xy 69.85 124.46) (xy 105.41 124.46))
+    (stroke (width 0) (type default) (color 0 0 0 0))
+  )
   (wire (pts (xy 194.31 110.49) (xy 73.66 110.49))
     (stroke (width 0) (type default) (color 0 0 0 0))
@@
   )
   (wire (pts (xy 160.02 88.9) (xy 171.45 88.9))
+    (stroke (width 0) (type default) (color 0 0 0 0))
+  )
+  (wire (pts (xy 69.85 119.38) (xy 76.2 119.38))
     (stroke (width 0) (type default) (color 0 0 0 0))
   )
@@
     )
   )
+  (global_label "phi1_2" (shape input) (at 69.85 124.46 180) (fields_autoplaced)
+    (effects (font (size 1.27 1.27)) (justify right))
+    (property "Intersheet References" "${INTERSHEET_REFS}" (id 0) (at 61.1474 124.3806 0)
+      (effects (font (size 1.27 1.27)) (justify right) hide)
+    )
+  )
   (global_label "~{Flag_SAVE->}" (shape output) (at 200.66 124.46 0) (fields_autoplaced)
     (effects (font (size 1.27 1.27)) (justify left))
@@
       (effects (font (size 1.27 1.27)) (justify right) hide)
     )
+  )
+  (global_label "phi2_2" (shape input) (at 69.85 119.38 180) (fields_autoplaced)
+    (effects (font (size 1.27 1.27)) (justify right))
+    (property "Intersheet References" "${INTERSHEET_REFS}" (id 0) (at 61.1474 119.3006 0)
+      (effects (font (size 1.27 1.27)) (justify right) hide)
+    )
