File: nlp-16a/Hardware/Instruction_decoder/POP_RET.kicad_sch (KiCad schematic)
At the start: 7 parts, among them U29 State_hold_unit, U30 State_hold_unit, U31 State_hold_unit, U32 State_hold_unit, U33 State_hold_unit, U34 State_hold_unit, U61 CD74HC00

Commit message: 基板設計 今日はとりあえずここまで
Parts:
- U29, U30, U31, U32, U33, U34: footprint (none) -> Connector_PinSocket_2.54mm:PinSocket_1x05_P2.54mm_Vertical
Connections:
- net OP5: now also U61.1; no longer U61.12
- net ~{->SP_INC_RET}: now also U61.5; no longer U61.1
- net ~{EXE_POP}: now also U61.8; no longer U61.6
- net at U30.3 (Q), U30.4 (LED), U61.13: now also U61.2; no longer U61.10
- new net: U61.11, U61.4
- new net: U61.10, U61.6, U61.9
- new net: U31.1 (D), U61.12, U61.3
Other:
- moved on the sheet: U61A, U61B, U61C, U61D
Changed lines of the file:
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@@
     (property "Reference" "U30" (id 0) (at 132.08 24.13 0))
     (property "Value" "State_hold_unit" (id 1) (at 132.08 26.67 0))
-    (property "Footprint" "" (id 2) (at 132.08 27.94 0)
+    (property "Footprint" "Connector_PinSocket_2.54mm:PinSocket_1x05_P2.54mm_Vertical" (id 2) (at 132.08 27.94 0)
       (effects (font (size 1.27 1.27)) hide)
     )
@@
     (pin "5")
   )
-  (symbol (lib_id "CD74HCXX:CD74HC00") (at 173.99 53.34 0) (mirror x) (unit 2)
+  (symbol (lib_id "CD74HCXX:CD74HC00") (at 156.21 53.34 0) (unit 2)
     (in_bom yes) (on_board yes)
-    (property "Reference" "U61" (id 0) (at 173.99 44.45 0))
-    (property "Value" "CD74HC00" (id 1) (at 173.99 46.99 0))
-    (property "Footprint" "Package_DIP:DIP-14_W7.62mm" (id 2) (at 173.99 59.69 0)
+    (property "Reference" "U61" (id 0) (at 156.21 44.45 0))
+    (property "Value" "CD74HC00" (id 1) (at 156.21 46.99 0))
+    (property "Footprint" "Package_DIP:DIP-14_W7.62mm" (id 2) (at 156.21 46.99 0)
       (effects (font (size 1.27 1.27)) hide)
     )
-    (property "Datasheet" "" (id 3) (at 168.91 53.34 0))
+    (property "Datasheet" "" (id 3) (at 151.13 53.34 0))
     (pin "14")
     (pin "7")
@@
     (property "Reference" "U29" (id 0) (at 100.33 24.13 0))
     (property "Value" "State_hold_unit" (id 1) (at 100.33 26.67 0))
-    (property "Footprint" "" (id 2) (at 100.33 27.94 0)
+    (property "Footprint" "Connector_PinSocket_2.54mm:PinSocket_1x05_P2.54mm_Vertical" (id 2) (at 100.33 27.94 0)
       (effects (font (size 1.27 1.27)) hide)
     )
@@
     (property "Reference" "U32" (id 0) (at 132.08 73.66 0))
     (property "Value" "State_hold_unit" (id 1) (at 132.08 76.2 0))
-    (property "Footprint" "" (id 2) (at 132.08 77.47 0)
+    (property "Footprint" "Connector_PinSocket_2.54mm:PinSocket_1x05_P2.54mm_Vertical" (id 2) (at 132.08 77.47 0)
       (effects (font (size 1.27 1.27)) hide)
     )
@@
     (property "Reference" "U33" (id 0) (at 100.33 93.98 0))
     (property "Value" "State_hold_unit" (id 1) (at 100.33 96.52 0))
-    (property "Footprint" "" (id 2) (at 100.33 97.79 0)
+    (property "Footprint" "Connector_PinSocket_2.54mm:PinSocket_1x05_P2.54mm_Vertical" (id 2) (at 100.33 97.79 0)
       (effects (font (size 1.27 1.27)) hide)
     )
@@
     (pin "5")
   )
-  (symbol (lib_id "CD74HCXX:CD74HC00") (at 102.87 50.8 0) (mirror x) (unit 3)
+  (symbol (lib_id "CD74HCXX:CD74HC00") (at 173.99 53.34 0) (unit 3)
+    (in_bom yes) (on_board yes)
+    (property "Reference" "U61" (id 0) (at 173.99 44.45 0))
+    (property "Value" "CD74HC00" (id 1) (at 173.99 46.99 0))
+    (property "Footprint" "Package_DIP:DIP-14_W7.62mm" (id 2) (at 173.99 46.99 0)
+      (effects (font (size 1.27 1.27)) hide)
+    )
+    (property "Datasheet" "" (id 3) (at 168.91 53.34 0))
+    (pin "14")
+    (pin "7")
+    (pin "1")
+    (pin "2")
+    (pin "3")
+    (pin "4")
+    (pin "5")
+    (pin "6")
+    (pin "10")
+    (pin "8")
+    (pin "9")
+    (pin "11")
+    (pin "12")
+    (pin "13")
+  )
+  (symbol (lib_id "CD74HCXX:CD74HC00") (at 102.87 50.8 0) (mirror x) (unit 4)
     (in_bom yes) (on_board yes)
     (property "Reference" "U61" (id 0) (at 102.87 41.91 0))
@@
     (pin "13")
   )
-  (symbol (lib_id "CD74HCXX:CD74HC00") (at 102.87 67.31 0) (mirror x) (unit 4)
+  (symbol (lib_id "State_hold_unit:State_hold_unit") (at 100.33 77.47 0) (unit 1)
+    (in_bom yes) (on_board yes) (fields_autoplaced)
+    (property "Reference" "U31" (id 0) (at 100.33 73.66 0))
+    (property "Value" "State_hold_unit" (id 1) (at 100.33 76.2 0))
+    (property "Footprint" "Connector_PinSocket_2.54mm:PinSocket_1x05_P2.54mm_Vertical" (id 2) (at 100.33 77.47 0)
+      (effects (font (size 1.27 1.27)) hide)
+    )
+    (property "Datasheet" "" (id 3) (at 100.33 77.47 0)
+      (effects (font (size 1.27 1.27)) hide)
+    )
+    (pin "1")
+    (pin "2")
+    (pin "3")
+    (pin "4")
+    (pin "5")
+  )
+  (symbol (lib_id "CD74HCXX:CD74HC00") (at 102.87 67.31 0) (mirror x) (unit 1)
     (in_bom yes) (on_board yes)
     (property "Reference" "U61" (id 0) (at 102.87 58.42 0))
@@
     (pin "13")
   )
-  (symbol (lib_id "State_hold_unit:State_hold_unit") (at 100.33 77.47 0) (unit 1)
-    (in_bom yes) (on_board yes) (fields_autoplaced)
-    (property "Reference" "U31" (id 0) (at 100.33 73.66 0))
-    (property "Value" "State_hold_unit" (id 1) (at 100.33 76.2 0))
-    (property "Footprint" "" (id 2) (at 100.33 77.47 0)
-      (effects (font (size 1.27 1.27)) hide)
-    )
-    (property "Datasheet" "" (id 3) (at 100.33 77.47 0)
-      (effects (font (size 1.27 1.27)) hide)
-    )
-    (pin "1")
-    (pin "2")
-    (pin "3")
-    (pin "4")
-    (pin "5")
-  )
-  (symbol (lib_id "CD74HCXX:CD74HC00") (at 156.21 53.34 0) (mirror x) (unit 1)
-    (in_bom yes) (on_board yes)
-    (property "Reference" "U61" (id 0) (at 156.21 44.45 0))
-    (property "Value" "CD74HC00" (id 1) (at 156.21 46.99 0))
-    (property "Footprint" "Package_DIP:DIP-14_W7.62mm" (id 2) (at 156.21 59.69 0)
-      (effects (font (size 1.27 1.27)) hide)
-    )
-    (property "Datasheet" "" (id 3) (at 151.13 53.34 0))
-    (pin "14")
-    (pin "7")
-    (pin "1")
-    (pin "2")
-    (pin "3")
-    (pin "4")
-    (pin "5")
-    (pin "6")
-    (pin "10")
-    (pin "8")
-    (pin "9")
-    (pin "11")
-    (pin "12")
-    (pin "13")
-  )
   (symbol (lib_id "State_hold_unit:State_hold_unit") (at 132.08 97.79 0) (unit 1)
     (in_bom yes) (on_board yes) (fields_autoplaced)
     (property "Reference" "U34" (id 0) (at 132.08 93.98 0))
     (property "Value" "State_hold_unit" (id 1) (at 132.08 96.52 0))
-    (property "Footprint" "" (id 2) (at 132.08 97.79 0)
+    (property "Footprint" "Connector_PinSocket_2.54mm:PinSocket_1x05_P2.54mm_Vertical" (id 2) (at 132.08 97.79 0)
       (effects (font (size 1.27 1.27)) hide)
     )

Commit message: 命令デコーダ完了！！
Connections:
- net phi1_1: now reaches U32.2 (G)
- net phi2_1: now reaches U31.2 (G)
- no-connect marks 6 -> 4
Changed lines of the file:
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@@
   (junction (at 110.49 86.36) (diameter 0) (color 0 0 0 0)
   )
-  (no_connect (at 90.17 86.36))
   (no_connect (at 121.92 36.83))
   (no_connect (at 121.92 106.68))
   (no_connect (at 90.17 36.83))
-  (no_connect (at 121.92 86.36))
   (no_connect (at 90.17 106.68))
   (wire (pts (xy 142.24 36.83) (xy 148.59 36.83))
     (stroke (width 0) (type default) (color 0 0 0 0))
   )
-  (wire (pts (xy 119.38 86.36) (xy 110.49 86.36))
-    (stroke (width 0) (type default) (color 0 0 0 0))
-  )
-  (wire (pts (xy 121.92 81.28) (xy 119.38 81.28))
+  (wire (pts (xy 118.11 86.36) (xy 110.49 86.36))
+    (stroke (width 0) (type default) (color 0 0 0 0))
+  )
+  (wire (pts (xy 121.92 81.28) (xy 118.11 81.28))
     (stroke (width 0) (type default) (color 0 0 0 0))
   )
@@
     (stroke (width 0) (type default) (color 0 0 0 0))
   )
-  (wire (pts (xy 119.38 81.28) (xy 119.38 86.36))
+  (wire (pts (xy 118.11 81.28) (xy 118.11 86.36))
     (stroke (width 0) (type default) (color 0 0 0 0))
   )
@@
     (stroke (width 0) (type default) (color 0 0 0 0))
   )
+  (wire (pts (xy 83.82 86.36) (xy 90.17 86.36))
+    (stroke (width 0) (type default) (color 0 0 0 0))
+  )
   (wire (pts (xy 110.49 106.68) (xy 111.76 106.68))
     (stroke (width 0) (type default) (color 0 0 0 0))
@@
     (stroke (width 0) (type default) (color 0 0 0 0))
   )
+  (wire (pts (xy 118.11 90.17) (xy 120.65 90.17))
+    (stroke (width 0) (type default) (color 0 0 0 0))
+  )
   (wire (pts (xy 119.38 36.83) (xy 110.49 36.83))
     (stroke (width 0) (type default) (color 0 0 0 0))
@@
     (stroke (width 0) (type default) (color 0 0 0 0))
   )
+  (wire (pts (xy 120.65 90.17) (xy 120.65 86.36))
+    (stroke (width 0) (type default) (color 0 0 0 0))
+  )
   (wire (pts (xy 87.63 101.6) (xy 87.63 95.25))
     (stroke (width 0) (type default) (color 0 0 0 0))
   )
+  (wire (pts (xy 120.65 86.36) (xy 121.92 86.36))
+    (stroke (width 0) (type default) (color 0 0 0 0))
+  )
   (wire (pts (xy 165.1 50.8) (xy 166.37 50.8))
     (stroke (width 0) (type default) (color 0 0 0 0))
   )
+  (global_label "phi1_1" (shape input) (at 118.11 90.17 180) (fields_autoplaced)
+    (effects (font (size 1.27 1.27)) (justify right))
+    (property "Intersheet References" "${INTERSHEET_REFS}" (id 0) (at 109.4074 90.0906 0)
+      (effects (font (size 1.27 1.27)) (justify right) hide)
+    )
+  )
   (global_label "~{EXE_POP}" (shape output) (at 181.61 53.34 0) (fields_autoplaced)
     (effects (font (size 1.27 1.27)) (justify left))
@@
     )
   )
+  (global_label "phi2_1" (shape input) (at 83.82 86.36 180) (fields_autoplaced)
+    (effects (font (size 1.27 1.27)) (justify right))
+    (property "Intersheet References" "${INTERSHEET_REFS}" (id 0) (at 75.1174 86.2806 0)
+      (effects (font (size 1.27 1.27)) (justify right) hide)
+    )
+  )
