File: nlp-16a/Hardware/Instruction_decoder/execute.kicad_sch (KiCad schematic)
At the start: 31 parts

Commit message: 命令デコーダ 不具合修正
Connections:
- net at U?.1, U?.3: now also U?.1; no longer U?.1 (D) (x2)
- net at U?.3: now also U?.1 (D); no longer U?.2
- net at U?.3: no longer U?.2
- net at U?.5 (~{Q}): now also U?.2; no longer U?.1
- net at U?.3 (Q), U?.4 (LED): no longer U?.1
- net at U?.5 (~{Q}): now also U?.2
Other:
- moved on the sheet: U?, U?A

Commit message: 命令デコーダ ロジック部の設計だいたい完了git statusgit statusやったぜ
Parts:
- removed U?: CD74HC00, Package_DIP:DIP-14_W7.62mm, symbol CD74HCXX:CD74HC00
- added U? (x3): CD74HC00, Package_DIP:DIP-14_W7.62mm, symbol CD74HCXX:CD74HC00
Connections:
- net GND: now also U?.7 (GND), U?.7 (GND), U?.7 (GND)
- net VCC: now also U?.14 (VCC), U?.14 (VCC), U?.14 (VCC)
- net WB: now reaches U?.2, U?.2, U?.3 (Q), U?.4 (LED)
- net at U?.3: now also U?.1 (D)
- net ~{->Flag_SET}: now reaches U?.2, U?.5 (~{Q})
- net ~{RA3}: now reaches U?.3 (Q)
- net ~{Flag_SET->}: now reaches U?.3 (Q)
- net ~{OP->}: now reaches U?.5 (~{Q})
- net ~{SP_INC_POP->}: now reaches U?.3 (Q)
- net ~{Acc}: now reaches U?.2, U?.5 (~{Q})
- net at U?.2, U?.3 (Q): now also U?.1
- net ~{RAM_LOAD}: now reaches U?.4 (LED), U?.5 (~{Q})
- net ~{Address_SET}: now reaches U?.2, U?.2, U?.4 (LED), U?.5 (~{Q})
- net ~{->SP_INC_POP}: now reaches U?.2, U?.5 (~{Q})
- new net: U?.2, U?.3
- new net: U?.1, U?.2, U?.3
- new net RAM_FETCH->: U?.1, U?.2
- new net ~{RAM_EXE->}: U?.3
- no-connect marks 9 -> 12
Other:
- note added: "LでRA3"
- note added: "SetAcc"
- note added: "SetFlag"
- note added: "Y Reg制御に対し， 内部処理モード/非内部処理モードの指定を行う．"

Commit message: アノテーションまで完了．基板設計に入る
Parts:
- removed U? (x3): CD74HC00, Package_DIP:DIP-14_W7.62mm, symbol CD74HCXX:CD74HC00
- gave numbers to parts that had none: 15
Connections:
- net END_EXE: now also U59.6; no longer U59.3
- net OP6: now also U55.12; no longer U55.1
- net OP7: now also U56.12, U57.5; no longer U56.1, U57.2
- net WB: now also U59.10, U59.13; no longer U59.2, U59.2
- net ~{->Flag_SET}: now also U56.5; no longer U56.2
- net ~{->SP_INC_POP}: now also U59.5; no longer U59.2
- net ~{EXE_POP}: now also U58.13; no longer U58.2
- net ~{EXE_PUSH}: now also U55.4; no longer U55.1
- net ~{PUSH_EXE}: now also U58.4; no longer U58.1
- net at U23.1 (D): now also U59.8; no longer U59.3
- net at U15.1 (D): now also U55.8; no longer U55.3
- net Y_Flag_sel: now reaches U17.4 (LED), U17.5 (~{Q}), U18.1 (D)
- net at U19.3 (Q), U19.4 (LED): now also U57.10, U57.13; no longer U57.2, U57.2
- net at U59.3: now also U59.12; no longer U59.1
- net at U17.1 (D): now also U56.8; no longer U56.3
- net at U55.3: now also U55.5; no longer U55.2
- net at U21.3 (Q): now also U21.4 (LED); no longer U58.2
- net at U19.1 (D): now also U56.6; no longer U56.3
- net at U57.3: now also U57.4; no longer U57.1
- net at U22.1 (D): now also U58.8; no longer U58.3
- net at U21.1 (D): now also U58.11; no longer U58.3
- net at U20.1 (D): now also U57.8; no longer U57.3
- net ~{Address_Y}: now reaches U20.3 (Q)
- net ~{Acc} renamed ~{Acc_Y}
- net ~{Address_SET}: no longer names the net of U20.4 (LED), U20.5 (~{Q}), U58.2
- net ~{Address_SET}: now also U58.5; no longer U58.2
- net ~{RAM_LOAD} renamed ~{RAM_LOAD->}
- net ~{RAM_LOAD->}: now also U58.10; no longer U21.4 (LED)
- new net: U59.11, U59.4, U59.9
- new net: U55.10, U55.13, U55.6
- new net: U55.11, U55.9, U56.1
- new net: U57.11, U57.9, U58.9
- new net: U57.12, U57.6
- new net: U56.10, U56.13, U56.3
- new net: U56.11, U56.4, U56.9
- new net: U58.12, U58.6
- no-connect marks 12 -> 11

Commit message: 基板設計 今日はとりあえずここまで
Parts:
- U15, U16, U17, U18, U19, U20, U21, U22, U23, U24: footprint (none) -> Connector_PinSocket_2.54mm:PinSocket_1x05_P2.54mm_Vertical
Connections:
- net OP7: now also U56.13; no longer U56.12
- net WB: now also U59.9; no longer U59.10
- net ~{EXE_POP}: now also U58.10; no longer U58.13
- net ~{EXE_PUSH}: now also U55.5; no longer U55.4
- net ~{RAM_LOAD->}: now also U58.13; no longer U58.10
- net at U59.11, U59.4: now also U59.10; no longer U59.9
- net at U55.13, U55.6: now also U55.9; no longer U55.10
- net at U55.11, U56.1: now also U55.10; no longer U55.9
- net at U57.12: now also U19.3 (Q), U19.4 (LED), U57.9; no longer U57.6
- net at U55.3: now also U55.4; no longer U55.5
- net at U56.11, U56.4: now also U56.10; no longer U56.9
- net at U58.8: now also U21.1 (D); no longer U22.1 (D)
- net at U58.11: now also U22.1 (D); no longer U21.1 (D)
- net at U58.12: now also U57.10, U57.11; no longer U58.6
- new net: U57.13, U57.6
- new net: U56.12, U56.3, U56.9
- new net: U58.6, U58.9
Other:
- moved on the sheet: U58C, U58D

Commit message: 基板設計 進捗
Connections:
- net ~{WB}: now reaches U22.5 (~{Q})
- net WB renamed ~{INTERNAL_Y}
- net ~{Acc_Y} renamed ~{AccWR}
- no-connect marks 11 -> 10
Changed lines of the file:
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@@
   (no_connect (at 149.86 34.29))
   (no_connect (at 175.26 74.93))
-  (no_connect (at 250.19 142.24))
   (no_connect (at 229.87 142.24))
   (no_connect (at 72.39 125.73))
@@
     (stroke (width 0) (type default) (color 0 0 0 0))
   )
+  (wire (pts (xy 250.19 142.24) (xy 255.27 142.24))
+    (stroke (width 0) (type default) (color 0 0 0 0))
+  )
   (wire (pts (xy 198.12 45.72) (xy 198.12 39.37))
     (stroke (width 0) (type default) (color 0 0 0 0))
@@
     (stroke (width 0) (type default) (color 0 0 0 0))
   )
+  (wire (pts (xy 252.73 137.16) (xy 255.27 137.16))
+    (stroke (width 0) (type default) (color 0 0 0 0))
+  )
   (wire (pts (xy 172.72 69.85) (xy 175.26 69.85))
     (stroke (width 0) (type default) (color 0 0 0 0))
@@
   )
   (wire (pts (xy 149.86 123.19) (xy 167.64 123.19))
-    (stroke (width 0) (type default) (color 0 0 0 0))
-  )
-  (wire (pts (xy 252.73 137.16) (xy 255.27 137.16))
     (stroke (width 0) (type default) (color 0 0 0 0))
   )
@@
     )
   )
-  (global_label "WB" (shape output) (at 255.27 137.16 0) (fields_autoplaced)
+  (global_label "~{WB}" (shape output) (at 255.27 142.24 0) (fields_autoplaced)
     (effects (font (size 1.27 1.27)) (justify left))
-    (property "Intersheet References" "${INTERSHEET_REFS}" (id 0) (at 260.4045 137.0806 0)
+    (property "Intersheet References" "${INTERSHEET_REFS}" (id 0) (at 260.4045 142.1606 0)
       (effects (font (size 1.27 1.27)) (justify left) hide)
     )
@@
     )
   )
-  (global_label "~{Acc_Y}" (shape output) (at 200.66 21.59 0) (fields_autoplaced)
+  (global_label "~{AccWR}" (shape output) (at 200.66 21.59 0) (fields_autoplaced)
     (effects (font (size 1.27 1.27)) (justify left))
-    (property "Intersheet References" "${INTERSHEET_REFS}" (id 0) (at 208.395 21.5106 0)
+    (property "Intersheet References" "${INTERSHEET_REFS}" (id 0) (at 209.0602 21.5106 0)
       (effects (font (size 1.27 1.27)) (justify left) hide)
     )
@@
       (effects (font (size 1.27 1.27)) (justify left) hide)
     )
+  )
+  (global_label "~{INTERNAL_Y}" (shape output) (at 255.27 137.16 0) (fields_autoplaced)
+    (effects (font (size 1.27 1.27)) (justify left))
+    (property "Intersheet References" "${INTERSHEET_REFS}" (id 0) (at 268.5083 137.0806 0)
+      (effects (font (size 1.27 1.27)) (justify left) hide)
+    )

Commit message: 命令デコーダ完了！！
Connections:
- net OP6: now also U59.2; no longer U59.1
- net OP7: now also U59.1; no longer U59.2
Changed lines of the file:
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@@
     )
   )
-  (global_label "OP7" (shape input) (at 52.07 177.8 180) (fields_autoplaced)
+  (global_label "OP7" (shape input) (at 52.07 182.88 180) (fields_autoplaced)
     (effects (font (size 1.27 1.27)) (justify right))
-    (property "Intersheet References" "${INTERSHEET_REFS}" (id 0) (at 45.8469 177.7206 0)
+    (property "Intersheet References" "${INTERSHEET_REFS}" (id 0) (at 45.8469 182.8006 0)
       (effects (font (size 1.27 1.27)) (justify right) hide)
     )
@@
     )
   )
-  (global_label "OP6" (shape input) (at 52.07 182.88 180) (fields_autoplaced)
+  (global_label "OP6" (shape input) (at 52.07 177.8 180) (fields_autoplaced)
     (effects (font (size 1.27 1.27)) (justify right))
-    (property "Intersheet References" "${INTERSHEET_REFS}" (id 0) (at 45.8469 182.8006 0)
+    (property "Intersheet References" "${INTERSHEET_REFS}" (id 0) (at 45.8469 177.7206 0)
       (effects (font (size 1.27 1.27)) (justify right) hide)
     )
