File: nlp-16a/Hardware/Instruction_decoder/Instruction_decoder.kicad_sch (KiCad schematic)
At the start: 0 parts

Commit message: 命令デコーダ ロジック部の設計だいたい完了git statusgit statusやったぜ
Other:
- added sheet control_signal (control_signal.kicad_sch)
- note added: "デコードシーケンス"
- note added: "制御信号生成"

Commit message: アノテーションまで完了．基板設計に入る
Other:
- added sheet sequence_start (sequence_start.kicad_sch)
- note added: "U1 - U48 -ステート保持ユニット(プレフィックスは分けるべきだったかもしれない) U49 - U64 -シーケンス，デコード U65- - 制御信号生成"
