File: nlp-16a/Hardware/Instruction_decoder/control_signal.kicad_sch (KiCad schematic)
At the start: 55 parts

Commit message: 命令デコーダ 軽微な修正
Parts:
- added U?: CD74HC00, Package_DIP:DIP-14_W7.62mm, symbol CD74HCXX:CD74HC00
Connections:
- net GND: now also U?.7 (GND)
- net VCC: now also U?.14 (VCC)
- net ~{DEC}: no longer U?.2
- net ~{SP_SET->}: now also U?.1, U?.2
- net at U?.1, U?.3: no longer U?.2
- net at U?.2, U?.3: now also U?.1, U?.2; no longer U?.1
- new net: U?.2, U?.3
Other:
- note added: "DECの抑制"
- note added: "INCの抑制"
Changed lines of the file:
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@@
   (junction (at 69.85 34.29) (diameter 0) (color 0 0 0 0)
   )
+  (junction (at 167.64 45.72) (diameter 0) (color 0 0 0 0)
+  )
   (junction (at 185.42 78.74) (diameter 0) (color 0 0 0 0)
   )
+  (junction (at 220.98 49.53) (diameter 0) (color 0 0 0 0)
+  )
   (junction (at 185.42 57.15) (diameter 0) (color 0 0 0 0)
   )
   (junction (at 87.63 156.21) (diameter 0) (color 0 0 0 0)
   )
+  (junction (at 167.64 49.53) (diameter 0) (color 0 0 0 0)
+  )
   (junction (at 185.42 121.92) (diameter 0) (color 0 0 0 0)
   )
@@
   (junction (at 52.07 43.18) (diameter 0) (color 0 0 0 0)
   )
-  (junction (at 238.76 35.56) (diameter 0) (color 0 0 0 0)
-  )
   (junction (at 52.07 105.41) (diameter 0) (color 0 0 0 0)
   )
@@
   (junction (at 185.42 92.71) (diameter 0) (color 0 0 0 0)
   )
-  (junction (at 256.54 68.58) (diameter 0) (color 0 0 0 0)
-  )
   (junction (at 87.63 128.27) (diameter 0) (color 0 0 0 0)
   )
@@
     (stroke (width 0) (type default) (color 0 0 0 0))
   )
+  (wire (pts (xy 222.25 54.61) (xy 220.98 54.61))
+    (stroke (width 0) (type default) (color 0 0 0 0))
+  )
   (wire (pts (xy 68.58 87.63) (xy 69.85 87.63))
     (stroke (width 0) (type default) (color 0 0 0 0))
@@
     (stroke (width 0) (type default) (color 0 0 0 0))
   )
+  (wire (pts (xy 220.98 49.53) (xy 222.25 49.53))
+    (stroke (width 0) (type default) (color 0 0 0 0))
+  )
   (wire (pts (xy 256.54 104.14) (xy 256.54 101.6))
     (stroke (width 0) (type default) (color 0 0 0 0))
@@
     (stroke (width 0) (type default) (color 0 0 0 0))
   )
+  (wire (pts (xy 218.44 38.1) (xy 222.25 38.1))
+    (stroke (width 0) (type default) (color 0 0 0 0))
+  )
   (wire (pts (xy 87.63 153.67) (xy 88.9 153.67))
     (stroke (width 0) (type default) (color 0 0 0 0))
@@
     (stroke (width 0) (type default) (color 0 0 0 0))
   )
+  (wire (pts (xy 257.81 66.04) (xy 256.54 66.04))
+    (stroke (width 0) (type default) (color 0 0 0 0))
+  )
   (wire (pts (xy 52.07 146.05) (xy 53.34 146.05))
     (stroke (width 0) (type default) (color 0 0 0 0))
@@
     (stroke (width 0) (type default) (color 0 0 0 0))
   )
-  (wire (pts (xy 220.98 35.56) (xy 220.98 38.1))
+  (wire (pts (xy 220.98 35.56) (xy 220.98 49.53))
     (stroke (width 0) (type default) (color 0 0 0 0))
   )
@@
     (stroke (width 0) (type default) (color 0 0 0 0))
   )
+  (wire (pts (xy 167.64 45.72) (xy 168.91 45.72))
+    (stroke (width 0) (type default) (color 0 0 0 0))
+  )
   (wire (pts (xy 186.69 59.69) (xy 185.42 59.69))
     (stroke (width 0) (type default) (color 0 0 0 0))
@@
     (stroke (width 0) (type default) (color 0 0 0 0))
   )
+  (wire (pts (xy 256.54 66.04) (xy 256.54 63.5))
+    (stroke (width 0) (type default) (color 0 0 0 0))
+  )
   (wire (pts (xy 53.34 151.13) (xy 52.07 151.13))
     (stroke (width 0) (type default) (color 0 0 0 0))
@@
     (stroke (width 0) (type default) (color 0 0 0 0))
   )
-  (wire (pts (xy 238.76 35.56) (xy 238.76 52.07))
-    (stroke (width 0) (type default) (color 0 0 0 0))
-  )
   (wire (pts (xy 52.07 105.41) (xy 52.07 107.95))
     (stroke (width 0) (type default) (color 0 0 0 0))
@@
     (stroke (width 0) (type default) (color 0 0 0 0))
   )
+  (wire (pts (xy 220.98 49.53) (xy 220.98 54.61))
+    (stroke (width 0) (type default) (color 0 0 0 0))
+  )
   (wire (pts (xy 203.2 87.63) (xy 204.47 87.63))
     (stroke (width 0) (type default) (color 0 0 0 0))
@@
     (stroke (width 0) (type default) (color 0 0 0 0))
   )
+  (wire (pts (xy 166.37 45.72) (xy 167.64 45.72))
+    (stroke (width 0) (type default) (color 0 0 0 0))
+  )
   (wire (pts (xy 220.98 85.09) (xy 220.98 87.63))
     (stroke (width 0) (type default) (color 0 0 0 0))
@@
     (stroke (width 0) (type default) (color 0 0 0 0))
   )
-  (wire (pts (xy 238.76 35.56) (xy 243.84 35.56))
+  (wire (pts (xy 237.49 35.56) (xy 243.84 35.56))
     (stroke (width 0) (type default) (color 0 0 0 0))
   )
@@
     (stroke (width 0) (type default) (color 0 0 0 0))
   )
-  (wire (pts (xy 222.25 38.1) (xy 220.98 38.1))
-    (stroke (width 0) (type default) (color 0 0 0 0))
-  )
   (wire (pts (xy 69.85 125.73) (xy 71.12 125.73))
     (stroke (width 0) (type default) (color 0 0 0 0))
@@
     (stroke (width 0) (type default) (color 0 0 0 0))
   )
-  (wire (pts (xy 168.91 45.72) (xy 166.37 45.72))
-    (stroke (width 0) (type default) (color 0 0 0 0))
-  )
   (wire (pts (xy 30.48 26.67) (xy 35.56 26.67))
     (stroke (width 0) (type default) (color 0 0 0 0))
@@
     (stroke (width 0) (type default) (color 0 0 0 0))
   )
+  (wire (pts (xy 256.54 63.5) (xy 167.64 63.5))
+    (stroke (width 0) (type default) (color 0 0 0 0))
+  )
   (wire (pts (xy 186.69 31.75) (xy 185.42 31.75))
     (stroke (width 0) (type default) (color 0 0 0 0))
@@
     (stroke (width 0) (type default) (color 0 0 0 0))
   )
-  (wire (pts (xy 256.54 66.04) (xy 257.81 66.04))
-    (stroke (width 0) (type default) (color 0 0 0 0))
-  )
   (wire (pts (xy 124.46 128.27) (xy 123.19 128.27))
     (stroke (width 0) (type default) (color 0 0 0 0))
@@
     (stroke (width 0) (type default) (color 0 0 0 0))
   )
-  (wire (pts (xy 238.76 52.07) (xy 240.03 52.07))
+  (wire (pts (xy 237.49 52.07) (xy 240.03 52.07))
     (stroke (width 0) (type default) (color 0 0 0 0))
   )
@@
     (stroke (width 0) (type default) (color 0 0 0 0))
   )
-  (wire (pts (xy 256.54 68.58) (xy 256.54 66.04))
-    (stroke (width 0) (type default) (color 0 0 0 0))
-  )
   (wire (pts (xy 87.63 52.07) (xy 87.63 49.53))
     (stroke (width 0) (type default) (color 0 0 0 0))
@@
     (stroke (width 0) (type default) (color 0 0 0 0))
   )
-  (wire (pts (xy 237.49 35.56) (xy 238.76 35.56))
-    (stroke (width 0) (type default) (color 0 0 0 0))
-  )
   (wire (pts (xy 87.63 49.53) (xy 88.9 49.53))
     (stroke (width 0) (type default) (color 0 0 0 0))
   )
+  (wire (pts (xy 167.64 45.72) (xy 167.64 49.53))
+    (stroke (width 0) (type default) (color 0 0 0 0))
+  )
+  (wire (pts (xy 167.64 49.53) (xy 218.44 49.53))
+    (stroke (width 0) (type default) (color 0 0 0 0))
+  )
   (wire (pts (xy 87.63 156.21) (xy 87.63 158.75))
     (stroke (width 0) (type default) (color 0 0 0 0))
@@
     (stroke (width 0) (type default) (color 0 0 0 0))
   )
+  (wire (pts (xy 218.44 49.53) (xy 218.44 38.1))
+    (stroke (width 0) (type default) (color 0 0 0 0))
+  )
   (wire (pts (xy 52.07 87.63) (xy 52.07 85.09))
     (stroke (width 0) (type default) (color 0 0 0 0))
@@
   )
   (wire (pts (xy 69.85 120.65) (xy 69.85 125.73))
+    (stroke (width 0) (type default) (color 0 0 0 0))
+  )
+  (wire (pts (xy 167.64 63.5) (xy 167.64 49.53))
     (stroke (width 0) (type default) (color 0 0 0 0))
   )
@@
   (text "BUS Dir逆転モード" (at 125.73 184.15 0)
     (effects (font (size 1.27 1.27)) (justify left bottom))
+  )
+  (text "INCの抑制" (at 214.63 63.5 180)
+    (effects (font (size 1.27 1.27)) (justify right bottom))
+  )
+  (text "DECの抑制" (at 214.63 49.53 180)
+    (effects (font (size 1.27 1.27)) (justify right bottom))
   )
   (text "A BUS 非内部処理" (at 16.51 100.33 0)
@@
     )
   )
+  (global_label "~{Address_SET}" (shape input) (at 142.24 189.23 180) (fields_autoplaced)
+    (effects (font (size 1.27 1.27)) (justify right))
+    (property "Intersheet References" "${INTERSHEET_REFS}" (id 0) (at 128.2155 189.1506 0)
+      (effects (font (size 1.27 1.27)) (justify right) hide)
+    )
+  )
   (global_label "~{IP_INC2->}" (shape input) (at 30.48 31.75 180) (fields_autoplaced)
     (effects (font (size 1.27 1.27)) (justify right))
@@
     )
   )
+  (global_label "~{IV_JMP->}" (shape input) (at 140.97 193.04 180) (fields_autoplaced)
+    (effects (font (size 1.27 1.27)) (justify right))
+    (property "Intersheet References" "${INTERSHEET_REFS}" (id 0) (at 129.0621 192.9606 0)
+      (effects (font (size 1.27 1.27)) (justify right) hide)
+    )
+  )
   (global_label "~{IP_Y}" (shape output) (at 139.7 78.74 0) (fields_autoplaced)
     (effects (font (size 1.27 1.27)) (justify left))
@@
     (pin "14")
     (pin "7")
+    (pin "1")
+    (pin "2")
+    (pin "3")
+    (pin "4")
+    (pin "5")
+    (pin "6")
+    (pin "10")
+    (pin "8")
+    (pin "9")
+    (pin "11")
+    (pin "12")
+    (pin "13")
+  )
+  (symbol (lib_id "CD74HCXX:CD74HC00") (at 229.87 52.07 0) (mirror x) (unit 1)
+    (in_bom yes) (on_board yes)
+    (property "Reference" "U?" (id 0) (at 229.87 43.18 0))
+    (property "Value" "CD74HC00" (id 1) (at 229.87 45.72 0))
+    (property "Footprint" "Package_DIP:DIP-14_W7.62mm" (id 2) (at 229.87 58.42 0)
+      (effects (font (size 1.27 1.27)) hide)
+    )
+    (property "Datasheet" "" (id 3) (at 224.79 52.07 0))
+    (pin "14")
+    (pin "7")

Commit message: アノテーションまで完了．基板設計に入る
Parts:
- added U37, U38: State_hold_unit, symbol State_hold_unit:State_hold_unit
- added unit 1 of U68
- added unit 2 of U68
- added unit 2 of U70
- added unit 3 of U70
- added unit 4 of U70
- added unit 1 of U71
- added unit 2 of U71
- added unit 3 of U81
- added unit 2 of U81
- added unit 1 of U81
- added U82: CD74HC00, Package_DIP:DIP-14_W7.62mm, symbol CD74HCXX:CD74HC00
- gave numbers to parts that had none: 17
Connections:
- net Fetch3->: now also U69.4; no longer U69.1
- net GND: now also U68.1, U68.2, U68.4, U68.5, U68.7 (GND), U68.7 (GND), U70.7 (GND), U70.7 (GND), U70.7 (GND), U71.7 (GND), U71.7 (GND), U81.1, U81.2, U81.4, U81.5, U81.7 (GND), U81.7 (GND), U81.7 (GND), U82.7 (GND), U82.7 (GND), U82.7 (GND), U82.7 (GND)
- net VCC: now also U68.14 (VCC), U68.14 (VCC), U70.14 (VCC), U70.14 (VCC), U70.14 (VCC), U71.14 (VCC), U71.14 (VCC), U81.14 (VCC), U81.14 (VCC), U81.14 (VCC), U82.14 (VCC), U82.14 (VCC), U82.14 (VCC), U82.14 (VCC)
- net ~{->Flag_Return}: now also U71.13; no longer U71.2
- net ~{->Flag_SET}: now also U71.12; no longer U71.1
- net ~{->IP_INC1}: now also U67.12; no longer U67.1
- net ~{->IP_SET}: now also U67.13; no longer U67.2
- net ~{->RAM_STORE}: now also U77.4; no longer U77.1
- net ~{Flag_Return->}: now also U72.12; no longer U72.1
- net ~{Flag_Y}: now also U71.8; no longer U71.3
- net ~{INTERNAL_ALU}: now also U70.12, U70.13
- net ~{IP_A}: now also U76.8; no longer U76.3
- net ~{IP_INC1->}: now also U65.13; no longer U65.2
- net ~{IP_INC2->}: now also U65.12; no longer U65.1
- net ~{IP_SAVE->}: now also U76.12; no longer U76.1
- net ~{IP_Y}: now also U76.6; no longer U76.3
- net ~{MEM_A}: now also U72.6; no longer U72.3
- net ~{MEM_Y}: now also U77.8; no longer U77.3
- net ~{OP->}: now also U70.5
- net ~{RA3}: now also U70.4, U71.1
- net ~{RAM_LOAD->}: now also U72.13; no longer U72.2
- net ~{RAM_STORE->}: now also U71.2
- net ~{SP_A}: now also U80.10, U80.6; no longer U80.2, U80.3
- net ~{SP_DEC_PUSH->}: now also U75.12; no longer U73.2
- net ~{SP_INC_POP->}: now also U75.13; no longer U75.2
- net ~{SP_INC_RET->}: now also U73.13; no longer U75.1
- net ~{SP_SET->}: now also U73.12, U78.9, U81.13; no longer U73.1, U78.1, U81.2
- net ~{SP_Y}: now also U79.8; no longer U79.3
- net at U76.1: now also U68.8; no longer U68.3
- net at U72.1: now also U69.8; no longer U69.3
- net at U72.2: now also U72.8; no longer U72.3
- net at U80.1, U80.2: now also U78.10, U78.6; no longer U78.2, U78.3
- net at U80.3: now also U80.13; no longer U80.2
- net ~{->IV_JMP} renamed ~{->IV_JMP/END_INT}
- removed net ~{DEC}: U78.3
- removed net ~{INC}: U81.3
- new net: U68.10, U68.11, U68.9
- new net: U82.10, U82.11
- new net: U37.1 (D), U82.12, U82.8
- new net: U82.13, U82.3
- new net: U75.10, U75.11, U75.9
- new net: U69.11, U69.5
- new net: U69.12, U69.13, U69.3
- new net: U69.10, U69.6, U69.9
- new net: U73.10, U73.11, U73.9
- new net: U77.12, U77.13, U77.3
- new net: U71.3, U71.4, U71.5
- new net: U67.10, U67.11, U67.9
- new net: U67.8, U68.13
- new net: U67.3, U67.4, U67.5
- new net: U80.8, U81.12
- new net: U81.8, U82.4, U82.5
- new net: U65.3, U65.4, U65.5
- new net: U65.10, U65.11, U65.9
- new net: U82.6, U82.9
- new net: U79.12, U79.13, U79.3
- new net: U72.3, U72.4, U72.5
- new net: U73.8, U78.4
- new net: U76.3, U76.4, U76.5
- new net: U73.3, U73.4, U73.5
- new net: U71.10, U71.11, U71.9
- new net: U78.11, U78.5
- new net: U78.12, U78.13, U78.3
- new net: U74.12, U74.13, U74.3
- new net: U77.10, U77.6, U77.9
- new net: U77.11, U77.5
- new net: U66.3, U66.4, U66.5
- new net: U66.6, U80.9
- new net: U72.10, U72.11, U72.9
- new net: U67.6, U68.12
- new net: U76.10, U76.11, U76.9
- new net: U66.8, U76.13
- new net: U79.11, U79.4
- new net: U74.8, U79.5
- new net: U79.10, U79.6, U79.9
- new net: U73.6, U74.4
- new net: U74.11, U74.5
- new net: U74.10, U74.6, U74.9
- new net: U70.9, U71.6
- new net: U65.8, U66.13, U66.2
- new net: U37.3 (Q), U37.4 (LED), U38.1 (D)
- new net: U80.11, U80.4, U80.5
- new net: U75.8, U80.12
- new net: U66.10, U66.11, U66.9
- new net: U65.6, U66.12
- new net: U70.10, U70.11
- new net INT_START: U82.1, U82.2
- new net ~{DEC_ALU}: U78.8
- new net ~{Fetch_END1}: U81.10
- new net ~{Fetch_END2}: U81.9
- new net ~{Fetch_Status}: U38.3 (Q), U38.4 (LED)
- new net ~{INC_ALU}: U81.11
- new net ~{INTERNAL_A}: U70.8
- new net ~{INTERNAL_Y}: U70.6
- no-connect marks 0 -> 8
Other:
- note added: "1サイクル分遅らせることでNOPの抑制のタイミングを調整"
- note added: "INT"
- note added: "POP/RET"
- note added: "PUSH"
- note added: "exe"
- note added: "fetch"
- note removed: "BUS Dir逆転モード"
- note removed: "コネクタへ直結可能"
- moved on the sheet: U70A, U71C, U71D, U77A, U77B, U77C, U77D
