File: nlp-16a/Hardware/Instruction_decoder/control_signal.kicad_sch (KiCad schematic)
At the start: 20 parts, among them U37 State_hold_unit, U38 State_hold_unit, U65 CD74HC00, U66 CD74HC00, U67 CD74HC00, U68 CD74HC00, U69 CD74HC00, U70 CD74HC00, U71 CD74HC00, U72 CD74HC00, U73 CD74HC00, U74 CD74HC00, U75 CD74HC00, U76 CD74HC00, U77 CD74HC00, U78 CD74HC00, U79 CD74HC00, U80 CD74HC00, U81 CD74HC00, U82 CD74HC00

Commit message: 基板設計 今日はとりあえずここまで
Parts:
- added unit 1 of U75
- added unit 2 of U75
- U37, U38: footprint (none) -> Connector_PinSocket_2.54mm:PinSocket_1x05_P2.54mm_Vertical
Connections:
- net GND: now also U75.1, U75.2, U75.4, U75.5, U75.7 (GND), U75.7 (GND)
- net VCC: now also U75.14 (VCC), U75.14 (VCC)
- net ~{->IP_INC1}: now also U67.13; no longer U67.12
- net ~{->IP_SET}: now also U67.12; no longer U67.13
- net ~{->RAM_STORE}: now also U77.5; no longer U77.4
- net ~{IP_INC3->}: now also U65.2; no longer U65.1
- net ~{IP_SET->}: now also U65.1; no longer U65.2
- net ~{OP->}: now also U70.4; no longer U70.5
- net ~{RA3}: now also U70.5; no longer U70.4
- net at U37.1 (D), U82.8: now also U82.13; no longer U82.12
- net at U82.3: now also U82.12; no longer U82.13
- net at U77.11: now also U77.4; no longer U77.5
- net at U74.4: now also U74.11; no longer U73.6
- net at U74.5: now also U73.6; no longer U74.11
- no-connect marks 8 -> 10
Changed lines of the file:
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@@
   (junction (at 123.19 39.37) (diameter 0) (color 0 0 0 0)
   )
+  (junction (at 245.11 25.4) (diameter 0) (color 0 0 0 0)
+  )
   (junction (at 52.07 120.65) (diameter 0) (color 0 0 0 0)
   )
@@
   (junction (at 87.63 36.83) (diameter 0) (color 0 0 0 0)
   )
+  (junction (at 265.43 25.4) (diameter 0) (color 0 0 0 0)
+  )
   (junction (at 123.19 125.73) (diameter 0) (color 0 0 0 0)
   )
@@
   (junction (at 256.54 54.61) (diameter 0) (color 0 0 0 0)
   )
+  (no_connect (at 283.21 22.86))
   (no_connect (at 257.81 162.56))
   (no_connect (at 237.49 162.56))
   (no_connect (at 125.73 100.33))
   (no_connect (at 146.05 100.33))
+  (no_connect (at 262.89 22.86))
   (no_connect (at 205.74 162.56))
   (no_connect (at 226.06 162.56))
@@
     (stroke (width 0) (type default) (color 0 0 0 0))
   )
+  (wire (pts (xy 265.43 25.4) (xy 267.97 25.4))
+    (stroke (width 0) (type default) (color 0 0 0 0))
+  )
   (wire (pts (xy 68.58 105.41) (xy 87.63 105.41))
     (stroke (width 0) (type default) (color 0 0 0 0))
@@
     (stroke (width 0) (type default) (color 0 0 0 0))
   )
+  (wire (pts (xy 265.43 20.32) (xy 267.97 20.32))
+    (stroke (width 0) (type default) (color 0 0 0 0))
+  )
   (wire (pts (xy 168.91 31.75) (xy 166.37 31.75))
     (stroke (width 0) (type default) (color 0 0 0 0))
@@
     (stroke (width 0) (type default) (color 0 0 0 0))
   )
+  (wire (pts (xy 245.11 25.4) (xy 245.11 20.32))
+    (stroke (width 0) (type default) (color 0 0 0 0))
+  )
   (wire (pts (xy 30.48 118.11) (xy 35.56 118.11))
     (stroke (width 0) (type default) (color 0 0 0 0))
@@
     (stroke (width 0) (type default) (color 0 0 0 0))
   )
+  (wire (pts (xy 265.43 26.67) (xy 265.43 25.4))
+    (stroke (width 0) (type default) (color 0 0 0 0))
+  )
   (wire (pts (xy 88.9 54.61) (xy 87.63 54.61))
     (stroke (width 0) (type default) (color 0 0 0 0))
@@
     (stroke (width 0) (type default) (color 0 0 0 0))
   )
+  (wire (pts (xy 245.11 26.67) (xy 245.11 25.4))
+    (stroke (width 0) (type default) (color 0 0 0 0))
+  )
   (wire (pts (xy 30.48 166.37) (xy 35.56 166.37))
     (stroke (width 0) (type default) (color 0 0 0 0))
@@
     (stroke (width 0) (type default) (color 0 0 0 0))
   )
+  (wire (pts (xy 245.11 20.32) (xy 247.65 20.32))
+    (stroke (width 0) (type default) (color 0 0 0 0))
+  )
   (wire (pts (xy 87.63 34.29) (xy 88.9 34.29))
     (stroke (width 0) (type default) (color 0 0 0 0))
@@
     (stroke (width 0) (type default) (color 0 0 0 0))
   )
+  (wire (pts (xy 245.11 25.4) (xy 247.65 25.4))
+    (stroke (width 0) (type default) (color 0 0 0 0))
+  )
   (wire (pts (xy 30.48 139.7) (xy 35.56 139.7))
     (stroke (width 0) (type default) (color 0 0 0 0))
@@
     (stroke (width 0) (type default) (color 0 0 0 0))
   )
+  (wire (pts (xy 265.43 25.4) (xy 265.43 20.32))
+    (stroke (width 0) (type default) (color 0 0 0 0))
+  )
   (wire (pts (xy 260.35 138.43) (xy 255.27 138.43))
     (stroke (width 0) (type default) (color 0 0 0 0))
@@
     (pin "13")
   )
-  (symbol (lib_id "CD74HCXX:CD74HC00") (at 247.65 121.92 0) (mirror x) (unit 4)
+  (symbol (lib_id "CD74HCXX:CD74HC00") (at 247.65 121.92 0) (unit 4)
     (in_bom yes) (on_board yes)
     (property "Reference" "U82" (id 0) (at 247.65 113.03 0))
     (property "Value" "CD74HC00" (id 1) (at 247.65 115.57 0))
-    (property "Footprint" "Package_DIP:DIP-14_W7.62mm" (id 2) (at 247.65 128.27 0)
+    (property "Footprint" "Package_DIP:DIP-14_W7.62mm" (id 2) (at 247.65 115.57 0)
       (effects (font (size 1.27 1.27)) hide)
     )
@@
     (pin "13")
   )
+  (symbol (lib_id "power:GND") (at 245.11 26.67 0) (unit 1)
+    (in_bom yes) (on_board yes) (fields_autoplaced)
+    (property "Reference" "#PWR020" (id 0) (at 245.11 33.02 0)
+      (effects (font (size 1.27 1.27)) hide)
+    )
+    (property "Value" "GND" (id 1) (at 245.11 31.75 0))
+    (property "Footprint" "" (id 2) (at 245.11 26.67 0)
+      (effects (font (size 1.27 1.27)) hide)
+    )
+    (property "Datasheet" "" (id 3) (at 245.11 26.67 0)
+      (effects (font (size 1.27 1.27)) hide)
+    )
+    (pin "1")
+  )
   (symbol (lib_id "CD74HCXX:CD74HC00") (at 176.53 43.18 0) (mirror x) (unit 4)
     (in_bom yes) (on_board yes)
@@
     (pin "13")
   )
-  (symbol (lib_id "CD74HCXX:CD74HC00") (at 43.18 73.66 0) (mirror x) (unit 4)
+  (symbol (lib_id "CD74HCXX:CD74HC00") (at 43.18 73.66 0) (unit 4)
     (in_bom yes) (on_board yes)
     (property "Reference" "U67" (id 0) (at 43.18 64.77 0))
     (property "Value" "CD74HC00" (id 1) (at 43.18 67.31 0))
-    (property "Footprint" "Package_DIP:DIP-14_W7.62mm" (id 2) (at 43.18 80.01 0)
+    (property "Footprint" "Package_DIP:DIP-14_W7.62mm" (id 2) (at 43.18 67.31 0)
       (effects (font (size 1.27 1.27)) hide)
     )
@@
     (pin "1")
   )
-  (symbol (lib_id "CD74HCXX:CD74HC00") (at 43.18 43.18 0) (mirror x) (unit 1)
+  (symbol (lib_id "CD74HCXX:CD74HC00") (at 43.18 43.18 0) (unit 1)
     (in_bom yes) (on_board yes)
     (property "Reference" "U65" (id 0) (at 43.18 34.29 0))
     (property "Value" "CD74HC00" (id 1) (at 43.18 36.83 0))
-    (property "Footprint" "Package_DIP:DIP-14_W7.62mm" (id 2) (at 43.18 49.53 0)
+    (property "Footprint" "Package_DIP:DIP-14_W7.62mm" (id 2) (at 43.18 36.83 0)
       (effects (font (size 1.27 1.27)) hide)
     )
@@
     (pin "13")
   )
-  (symbol (lib_id "CD74HCXX:CD74HC00") (at 78.74 149.86 0) (mirror x) (unit 2)
+  (symbol (lib_id "CD74HCXX:CD74HC00") (at 78.74 149.86 0) (unit 2)
     (in_bom yes) (on_board yes)
     (property "Reference" "U77" (id 0) (at 78.74 140.97 0))
     (property "Value" "CD74HC00" (id 1) (at 78.74 143.51 0))
-    (property "Footprint" "Package_DIP:DIP-14_W7.62mm" (id 2) (at 78.74 156.21 0)
+    (property "Footprint" "Package_DIP:DIP-14_W7.62mm" (id 2) (at 78.74 143.51 0)
       (effects (font (size 1.27 1.27)) hide)
     )
@@
     (pin "13")
   )
+  (symbol (lib_id "CD74HCXX:CD74HC00") (at 255.27 22.86 0) (mirror x) (unit 1)
+    (in_bom yes) (on_board yes)
+    (property "Reference" "U75" (id 0) (at 255.27 13.97 0))
+    (property "Value" "CD74HC00" (id 1) (at 255.27 16.51 0))
+    (property "Footprint" "Package_DIP:DIP-14_W7.62mm" (id 2) (at 255.27 29.21 0)
+      (effects (font (size 1.27 1.27)) hide)
+    )
+    (property "Datasheet" "" (id 3) (at 250.19 22.86 0))
+    (pin "14")
+    (pin "7")
+    (pin "1")
+    (pin "2")
+    (pin "3")
+    (pin "4")
+    (pin "5")
+    (pin "6")
+    (pin "10")
+    (pin "8")
+    (pin "9")
+    (pin "11")
+    (pin "12")
+    (pin "13")
+  )
   (symbol (lib_id "CD74HCXX:CD74HC00") (at 78.74 81.28 0) (mirror x) (unit 4)
     (in_bom yes) (on_board yes)
@@
     (pin "13")
   )
-  (symbol (lib_id "CD74HCXX:CD74HC00") (at 212.09 85.09 0) (mirror x) (unit 2)
+  (symbol (lib_id "CD74HCXX:CD74HC00") (at 212.09 85.09 0) (unit 2)
     (in_bom yes) (on_board yes)
     (property "Reference" "U74" (id 0) (at 212.09 76.2 0))
     (property "Value" "CD74HC00" (id 1) (at 212.09 78.74 0))
-    (property "Footprint" "Package_DIP:DIP-14_W7.62mm" (id 2) (at 212.09 91.44 0)
+    (property "Footprint" "Package_DIP:DIP-14_W7.62mm" (id 2) (at 212.09 78.74 0)
       (effects (font (size 1.27 1.27)) hide)
     )
@@
     (property "Reference" "U37" (id 0) (at 215.9 149.86 0))
     (property "Value" "State_hold_unit" (id 1) (at 215.9 152.4 0))
-    (property "Footprint" "" (id 2) (at 215.9 153.67 0)
+    (property "Footprint" "Connector_PinSocket_2.54mm:PinSocket_1x05_P2.54mm_Vertical" (id 2) (at 215.9 153.67 0)
       (effects (font (size 1.27 1.27)) hide)
     )
@@
     (pin "1")
   )
-  (symbol (lib_id "CD74HCXX:CD74HC00") (at 138.43 177.8 0) (mirror x) (unit 2)
+  (symbol (lib_id "CD74HCXX:CD74HC00") (at 138.43 177.8 0) (unit 2)
     (in_bom yes) (on_board yes)
     (property "Reference" "U70" (id 0) (at 138.43 168.91 0))
     (property "Value" "CD74HC00" (id 1) (at 138.43 171.45 0))
-    (property "Footprint" "Package_DIP:DIP-14_W7.62mm" (id 2) (at 138.43 184.15 0)
+    (property "Footprint" "Package_DIP:DIP-14_W7.62mm" (id 2) (at 138.43 171.45 0)
       (effects (font (size 1.27 1.27)) hide)
     )
@@
     (pin "13")
   )
+  (symbol (lib_id "CD74HCXX:CD74HC00") (at 275.59 22.86 0) (mirror x) (unit 2)
+    (in_bom yes) (on_board yes)
+    (property "Reference" "U75" (id 0) (at 275.59 13.97 0))
+    (property "Value" "CD74HC00" (id 1) (at 275.59 16.51 0))
+    (property "Footprint" "Package_DIP:DIP-14_W7.62mm" (id 2) (at 275.59 29.21 0)
+      (effects (font (size 1.27 1.27)) hide)
+    )
+    (property "Datasheet" "" (id 3) (at 270.51 22.86 0))
+    (pin "14")
+    (pin "7")
+    (pin "1")
+    (pin "2")
+    (pin "3")
+    (pin "4")
+    (pin "5")
+    (pin "6")
+    (pin "10")
+    (pin "8")
+    (pin "9")
+    (pin "11")
+    (pin "12")
+    (pin "13")
+  )
   (symbol (lib_id "CD74HCXX:CD74HC00") (at 229.87 85.09 0) (mirror x) (unit 3)
     (in_bom yes) (on_board yes)
@@
     (pin "13")
   )
+  (symbol (lib_id "power:GND") (at 265.43 26.67 0) (unit 1)
+    (in_bom yes) (on_board yes) (fields_autoplaced)
+    (property "Reference" "#PWR021" (id 0) (at 265.43 33.02 0)
+      (effects (font (size 1.27 1.27)) hide)
+    )
+    (property "Value" "GND" (id 1) (at 265.43 31.75 0))
+    (property "Footprint" "" (id 2) (at 265.43 26.67 0)
+      (effects (font (size 1.27 1.27)) hide)
+    )
+    (property "Datasheet" "" (id 3) (at 265.43 26.67 0)
+      (effects (font (size 1.27 1.27)) hide)
+    )
+    (pin "1")
+  )
   (symbol (lib_id "CD74HCXX:CD74HC00") (at 247.65 138.43 0) (mirror x) (unit 3)
     (in_bom yes) (on_board yes)
@@
     (property "Reference" "U38" (id 0) (at 247.65 149.86 0))
     (property "Value" "State_hold_unit" (id 1) (at 247.65 152.4 0))
-    (property "Footprint" "" (id 2) (at 247.65 153.67 0)
+    (property "Footprint" "Connector_PinSocket_2.54mm:PinSocket_1x05_P2.54mm_Vertical" (id 2) (at 247.65 153.67 0)
       (effects (font (size 1.27 1.27)) hide)
     )

Commit message: 基板設計 進捗
Connections:
- net ~{OP->}: no longer U70.4
- net ~{RA3}: no longer U70.5
- net at U80.3: now also U80.12; no longer U80.13
- net at U75.8: now also U80.13; no longer U80.12
- net ~{INTERNAL_Y} renamed Acc_Y
- new net ~{AccWR}: U70.4
- new net ~{WB}: U70.5
Changed lines of the file:
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@@
     )
   )
-  (global_label "~{RA3}" (shape input) (at 128.27 180.34 180) (fields_autoplaced)
-    (effects (font (size 1.27 1.27)) (justify right))
-    (property "Intersheet References" "${INTERSHEET_REFS}" (id 0) (at 122.2888 180.2606 0)
+  (global_label "~{AccWR}" (shape input) (at 128.27 175.26 180) (fields_autoplaced)
+    (effects (font (size 1.27 1.27)) (justify right))
+    (property "Intersheet References" "${INTERSHEET_REFS}" (id 0) (at 119.8698 175.1806 0)
       (effects (font (size 1.27 1.27)) (justify right) hide)
     )
@@
     )
   )
-  (global_label "~{INTERNAL_Y}" (shape output) (at 149.86 177.8 0) (fields_autoplaced)
+  (global_label "Acc_Y" (shape output) (at 149.86 177.8 0) (fields_autoplaced)
     (effects (font (size 1.27 1.27)) (justify left))
-    (property "Intersheet References" "${INTERSHEET_REFS}" (id 0) (at 163.0983 177.7206 0)
+    (property "Intersheet References" "${INTERSHEET_REFS}" (id 0) (at 157.595 177.7206 0)
       (effects (font (size 1.27 1.27)) (justify left) hide)
     )
@@
     )
   )
-  (global_label "~{OP->}" (shape input) (at 128.27 175.26 180) (fields_autoplaced)
-    (effects (font (size 1.27 1.27)) (justify right))
-    (property "Intersheet References" "${INTERSHEET_REFS}" (id 0) (at 120.1117 175.1806 0)
+  (global_label "~{WB}" (shape input) (at 128.27 180.34 180) (fields_autoplaced)
+    (effects (font (size 1.27 1.27)) (justify right))
+    (property "Intersheet References" "${INTERSHEET_REFS}" (id 0) (at 123.1355 180.2606 0)
       (effects (font (size 1.27 1.27)) (justify right) hide)
     )
@@
     (pin "13")
   )
-  (symbol (lib_id "CD74HCXX:CD74HC00") (at 247.65 54.61 0) (mirror x) (unit 4)
+  (symbol (lib_id "CD74HCXX:CD74HC00") (at 247.65 54.61 0) (unit 4)
     (in_bom yes) (on_board yes)
     (property "Reference" "U80" (id 0) (at 247.65 45.72 0))
     (property "Value" "CD74HC00" (id 1) (at 247.65 48.26 0))
-    (property "Footprint" "Package_DIP:DIP-14_W7.62mm" (id 2) (at 247.65 60.96 0)
-      (effects (font (size 1.27 1.27)) hide)
-    )
+    (property "Footprint" "Package_DIP:DIP-14_W7.62mm" (id 2) (at 247.65 48.26 0)
+      (effects (font (size 1.27 1.27)) hide)
+    )

Commit message: 命令デコーダ完了！！
Parts:
- added D3: LED, LED_THT:LED_D3.0mm, symbol Device:LED
- added R3: R, Resistor_SMD:R_0603_1608Metric_Pad0.98x0.95mm_HandSolder, symbol Device:R
Connections:
- net GND: now also R3.2
- net phi2_2: now reaches U37.2 (G)
- net phi1_2: now reaches U38.2 (G)
- net at U38.5 (~{Q}): now also D3.2 (A)
- new net: D3.1 (K), R3.1
- no-connect marks 10 -> 7
Changed lines of the file:
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@@
   )
   (no_connect (at 283.21 22.86))
-  (no_connect (at 257.81 162.56))
-  (no_connect (at 237.49 162.56))
   (no_connect (at 125.73 100.33))
   (no_connect (at 146.05 100.33))
   (no_connect (at 262.89 22.86))
-  (no_connect (at 205.74 162.56))
   (no_connect (at 226.06 162.56))
   (no_connect (at 168.91 128.27))
@@
     (stroke (width 0) (type default) (color 0 0 0 0))
   )
+  (wire (pts (xy 281.94 161.29) (xy 281.94 163.83))
+    (stroke (width 0) (type default) (color 0 0 0 0))
+  )
   (polyline (pts (xy 105.41 92.71) (xy 105.41 67.31))
     (stroke (width 0) (type default) (color 0 0 0 0))
@@
     (stroke (width 0) (type default) (color 0 0 0 0))
   )
+  (wire (pts (xy 278.13 161.29) (xy 281.94 161.29))
+    (stroke (width 0) (type default) (color 0 0 0 0))
+  )
   (polyline (pts (xy 31.75 17.78) (xy 104.14 17.78))
     (stroke (width 0) (type default) (color 0 0 0 0))
@@
     (stroke (width 0) (type default) (color 0 0 0 0))
   )
+  (wire (pts (xy 257.81 161.29) (xy 261.62 161.29))
+    (stroke (width 0) (type default) (color 0 0 0 0))
+  )
   (wire (pts (xy 184.15 78.74) (xy 185.42 78.74))
     (stroke (width 0) (type default) (color 0 0 0 0))
@@
     (stroke (width 0) (type default) (color 0 0 0 0))
   )
+  (wire (pts (xy 269.24 161.29) (xy 270.51 161.29))
+    (stroke (width 0) (type default) (color 0 0 0 0))
+  )
   (wire (pts (xy 52.07 43.18) (xy 52.07 40.64))
     (stroke (width 0) (type default) (color 0 0 0 0))
@@
     (stroke (width 0) (type default) (color 0 0 0 0))
   )
-  (wire (pts (xy 269.24 157.48) (xy 257.81 157.48))
+  (wire (pts (xy 257.81 157.48) (xy 269.24 157.48))
     (stroke (width 0) (type default) (color 0 0 0 0))
   )
@@
     (stroke (width 0) (type default) (color 0 0 0 0))
   )
+  (wire (pts (xy 257.81 162.56) (xy 257.81 161.29))
+    (stroke (width 0) (type default) (color 0 0 0 0))
+  )
   (wire (pts (xy 69.85 120.65) (xy 69.85 125.73))
     (stroke (width 0) (type default) (color 0 0 0 0))
@@
     (stroke (width 0) (type default) (color 0 0 0 0))
   )
+  (wire (pts (xy 199.39 162.56) (xy 205.74 162.56))
+    (stroke (width 0) (type default) (color 0 0 0 0))
+  )
   (wire (pts (xy 30.48 193.04) (xy 35.56 193.04))
     (stroke (width 0) (type default) (color 0 0 0 0))
@@
     )
   )
+  (global_label "phi2_2" (shape input) (at 199.39 162.56 180) (fields_autoplaced)
+    (effects (font (size 1.27 1.27)) (justify right))
+    (property "Intersheet References" "${INTERSHEET_REFS}" (id 0) (at 190.6874 162.4806 0)
+      (effects (font (size 1.27 1.27)) (justify right) hide)
+    )
+  )
   (global_label "~{->RAM_STORE}" (shape input) (at 30.48 152.4 180) (fields_autoplaced)
     (effects (font (size 1.27 1.27)) (justify right))
@@
     )
   )
+  (global_label "phi1_2" (shape input) (at 237.49 162.56 180) (fields_autoplaced)
+    (effects (font (size 1.27 1.27)) (justify right))
+    (property "Intersheet References" "${INTERSHEET_REFS}" (id 0) (at 228.7874 162.4806 0)
+      (effects (font (size 1.27 1.27)) (justify right) hide)
+    )
+  )
   (global_label "~{Flag_SET->}" (shape input) (at 30.48 161.29 180) (fields_autoplaced)
     (effects (font (size 1.27 1.27)) (justify right))
@@
     (pin "13")
   )
+  (symbol (lib_id "Device:LED") (at 265.43 161.29 180) (unit 1)
+    (in_bom yes) (on_board yes)
+    (property "Reference" "D3" (id 0) (at 267.97 163.83 0))
+    (property "Value" "LED" (id 1) (at 262.89 163.83 0))
+    (property "Footprint" "LED_THT:LED_D3.0mm" (id 2) (at 265.43 161.29 0)
+      (effects (font (size 1.27 1.27)) hide)
+    )
+    (property "Datasheet" "~" (id 3) (at 265.43 161.29 0)
+      (effects (font (size 1.27 1.27)) hide)
+    )
+    (pin "1")
+    (pin "2")
+  )
   (symbol (lib_id "CD74HCXX:CD74HC00") (at 43.18 105.41 0) (mirror x) (unit 4)
     (in_bom yes) (on_board yes)
@@
     (pin "13")
   )
+  (symbol (lib_id "Device:R") (at 274.32 161.29 90) (unit 1)
+    (in_bom yes) (on_board yes)
+    (property "Reference" "R3" (id 0) (at 273.05 163.83 90))
+    (property "Value" "R" (id 1) (at 275.59 163.83 90))
+    (property "Footprint" "Resistor_SMD:R_0603_1608Metric_Pad0.98x0.95mm_HandSolder" (id 2) (at 274.32 163.068 90)
+      (effects (font (size 1.27 1.27)) hide)
+    )
+    (property "Datasheet" "~" (id 3) (at 274.32 161.29 0)
+      (effects (font (size 1.27 1.27)) hide)
+    )
+    (pin "1")
+    (pin "2")
+  )
   (symbol (lib_id "power:GND") (at 128.27 104.14 0) (unit 1)
     (in_bom yes) (on_board yes) (fields_autoplaced)
@@
     (pin "13")
   )
+  (symbol (lib_id "power:GND") (at 281.94 163.83 0) (unit 1)
+    (in_bom yes) (on_board yes)
+    (property "Reference" "#PWR024" (id 0) (at 281.94 170.18 0)
+      (effects (font (size 1.27 1.27)) hide)
+    )
+    (property "Value" "GND" (id 1) (at 279.4 165.1 0))
+    (property "Footprint" "" (id 2) (at 281.94 163.83 0)
+      (effects (font (size 1.27 1.27)) hide)
+    )
+    (property "Datasheet" "" (id 3) (at 281.94 163.83 0)
+      (effects (font (size 1.27 1.27)) hide)
+    )
+    (pin "1")
+  )
   (symbol (lib_id "CD74HCXX:CD74HC00") (at 265.43 104.14 0) (mirror x) (unit 3)
