File: nlp-16a/Hardware/Instruction_decoder/control_signal.kicad_sch (KiCad schematic)
At the start: 22 parts, among them U37 State_hold_unit, U38 State_hold_unit, U65 CD74HC00, U66 CD74HC00, U67 CD74HC00, U68 CD74HC00, U69 CD74HC00, U70 CD74HC00, U71 CD74HC00, U72 CD74HC00, U73 CD74HC00, U74 CD74HC00, U75 CD74HC00, U76 CD74HC00, U77 CD74HC00, U78 CD74HC00, U79 CD74HC00, U80 CD74HC00, U81 CD74HC00, U82 CD74HC00

Commit message: 命令デコーダ修正
Connections:
- net ~{SP_DEC_PUSH->}: now also U73.13; no longer U75.12
- net ~{SP_INC_RET->}: now also U75.12; no longer U73.13
- net Fetch_Status: now reaches D3.2 (A), U38.5 (~{Q})
Changed lines of the file:
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@@
   (junction (at 87.63 52.07) (diameter 0) (color 0 0 0 0)
   )
+  (junction (at 52.07 73.66) (diameter 0) (color 0 0 0 0)
+  )
+  (junction (at 185.42 106.68) (diameter 0) (color 0 0 0 0)
+  )
+  (junction (at 87.63 36.83) (diameter 0) (color 0 0 0 0)
+  )
+  (junction (at 265.43 25.4) (diameter 0) (color 0 0 0 0)
+  )
+  (junction (at 123.19 125.73) (diameter 0) (color 0 0 0 0)
+  )
+  (junction (at 52.07 87.63) (diameter 0) (color 0 0 0 0)
+  )
+  (junction (at 185.42 43.18) (diameter 0) (color 0 0 0 0)
+  )
+  (junction (at 69.85 34.29) (diameter 0) (color 0 0 0 0)
+  )
+  (junction (at 167.64 45.72) (diameter 0) (color 0 0 0 0)
+  )
+  (junction (at 128.27 102.87) (diameter 0) (color 0 0 0 0)
+  )
+  (junction (at 185.42 78.74) (diameter 0) (color 0 0 0 0)
+  )
+  (junction (at 218.44 140.97) (diameter 0) (color 0 0 0 0)
+  )
+  (junction (at 220.98 49.53) (diameter 0) (color 0 0 0 0)
+  )
+  (junction (at 185.42 57.15) (diameter 0) (color 0 0 0 0)
+  )
+  (junction (at 87.63 149.86) (diameter 0) (color 0 0 0 0)
+  )
+  (junction (at 167.64 49.53) (diameter 0) (color 0 0 0 0)
+  )
+  (junction (at 147.32 163.83) (diameter 0) (color 0 0 0 0)
+  )
+  (junction (at 260.35 161.29) (diameter 0) (color 0 0 0 0)
+  )
+  (junction (at 151.13 130.81) (diameter 0) (color 0 0 0 0)
+  )
+  (junction (at 52.07 29.21) (diameter 0) (color 0 0 0 0)
+  )
+  (junction (at 185.42 29.21) (diameter 0) (color 0 0 0 0)
+  )
+  (junction (at 52.07 142.24) (diameter 0) (color 0 0 0 0)
+  )
+  (junction (at 52.07 172.72) (diameter 0) (color 0 0 0 0)
+  )
+  (junction (at 52.07 43.18) (diameter 0) (color 0 0 0 0)
+  )
+  (junction (at 52.07 105.41) (diameter 0) (color 0 0 0 0)
+  )
+  (junction (at 220.98 35.56) (diameter 0) (color 0 0 0 0)
+  )
+  (junction (at 260.35 138.43) (diameter 0) (color 0 0 0 0)
+  )
+  (junction (at 185.42 92.71) (diameter 0) (color 0 0 0 0)
+  )
+  (junction (at 87.63 128.27) (diameter 0) (color 0 0 0 0)
+  )
   (junction (at 257.81 157.48) (diameter 0) (color 0 0 0 0)
-  )
-  (junction (at 52.07 73.66) (diameter 0) (color 0 0 0 0)
-  )
-  (junction (at 185.42 106.68) (diameter 0) (color 0 0 0 0)
-  )
-  (junction (at 87.63 36.83) (diameter 0) (color 0 0 0 0)
-  )
-  (junction (at 265.43 25.4) (diameter 0) (color 0 0 0 0)
-  )
-  (junction (at 123.19 125.73) (diameter 0) (color 0 0 0 0)
-  )
-  (junction (at 52.07 87.63) (diameter 0) (color 0 0 0 0)
-  )
-  (junction (at 185.42 43.18) (diameter 0) (color 0 0 0 0)
-  )
-  (junction (at 69.85 34.29) (diameter 0) (color 0 0 0 0)
-  )
-  (junction (at 167.64 45.72) (diameter 0) (color 0 0 0 0)
-  )
-  (junction (at 128.27 102.87) (diameter 0) (color 0 0 0 0)
-  )
-  (junction (at 185.42 78.74) (diameter 0) (color 0 0 0 0)
-  )
-  (junction (at 218.44 140.97) (diameter 0) (color 0 0 0 0)
-  )
-  (junction (at 220.98 49.53) (diameter 0) (color 0 0 0 0)
-  )
-  (junction (at 185.42 57.15) (diameter 0) (color 0 0 0 0)
-  )
-  (junction (at 87.63 149.86) (diameter 0) (color 0 0 0 0)
-  )
-  (junction (at 167.64 49.53) (diameter 0) (color 0 0 0 0)
-  )
-  (junction (at 147.32 163.83) (diameter 0) (color 0 0 0 0)
-  )
-  (junction (at 151.13 130.81) (diameter 0) (color 0 0 0 0)
-  )
-  (junction (at 52.07 29.21) (diameter 0) (color 0 0 0 0)
-  )
-  (junction (at 185.42 29.21) (diameter 0) (color 0 0 0 0)
-  )
-  (junction (at 52.07 142.24) (diameter 0) (color 0 0 0 0)
-  )
-  (junction (at 52.07 172.72) (diameter 0) (color 0 0 0 0)
-  )
-  (junction (at 52.07 43.18) (diameter 0) (color 0 0 0 0)
-  )
-  (junction (at 52.07 105.41) (diameter 0) (color 0 0 0 0)
-  )
-  (junction (at 220.98 35.56) (diameter 0) (color 0 0 0 0)
-  )
-  (junction (at 260.35 138.43) (diameter 0) (color 0 0 0 0)
-  )
-  (junction (at 185.42 92.71) (diameter 0) (color 0 0 0 0)
-  )
-  (junction (at 87.63 128.27) (diameter 0) (color 0 0 0 0)
   )
   (junction (at 87.63 81.28) (diameter 0) (color 0 0 0 0)
@@
     (stroke (width 0) (type default) (color 0 0 0 0))
   )
+  (wire (pts (xy 260.35 156.21) (xy 260.35 161.29))
+    (stroke (width 0) (type default) (color 0 0 0 0))
+  )
   (wire (pts (xy 52.07 40.64) (xy 53.34 40.64))
     (stroke (width 0) (type default) (color 0 0 0 0))
@@
     (stroke (width 0) (type default) (color 0 0 0 0))
   )
+  (wire (pts (xy 260.35 161.29) (xy 261.62 161.29))
+    (stroke (width 0) (type default) (color 0 0 0 0))
+  )
   (wire (pts (xy 257.81 157.48) (xy 257.81 160.02))
     (stroke (width 0) (type default) (color 0 0 0 0))
@@
     (stroke (width 0) (type default) (color 0 0 0 0))
   )
-  (wire (pts (xy 257.81 161.29) (xy 261.62 161.29))
+  (wire (pts (xy 257.81 161.29) (xy 260.35 161.29))
     (stroke (width 0) (type default) (color 0 0 0 0))
   )
@@
     (stroke (width 0) (type default) (color 0 0 0 0))
   )
+  (wire (pts (xy 269.24 153.67) (xy 257.81 153.67))
+    (stroke (width 0) (type default) (color 0 0 0 0))
+  )
   (wire (pts (xy 69.85 78.74) (xy 71.12 78.74))
     (stroke (width 0) (type default) (color 0 0 0 0))
@@
     (stroke (width 0) (type default) (color 0 0 0 0))
   )
-  (wire (pts (xy 257.81 157.48) (xy 269.24 157.48))
-    (stroke (width 0) (type default) (color 0 0 0 0))
-  )
   (polyline (pts (xy 168.91 100.33) (xy 236.22 100.33))
     (stroke (width 0) (type default) (color 0 0 0 0))
@@
     (stroke (width 0) (type default) (color 0 0 0 0))
   )
+  (wire (pts (xy 257.81 153.67) (xy 257.81 157.48))
+    (stroke (width 0) (type default) (color 0 0 0 0))
+  )
   (wire (pts (xy 123.19 123.19) (xy 124.46 123.19))
     (stroke (width 0) (type default) (color 0 0 0 0))
@@
   )
   (wire (pts (xy 256.54 68.58) (xy 256.54 71.12))
+    (stroke (width 0) (type default) (color 0 0 0 0))
+  )
+  (wire (pts (xy 269.24 156.21) (xy 260.35 156.21))
     (stroke (width 0) (type default) (color 0 0 0 0))
   )
@@
     )
   )
+  (global_label "Fetch_Status" (shape output) (at 269.24 156.21 0) (fields_autoplaced)
+    (effects (font (size 1.27 1.27)) (justify left))
+    (property "Intersheet References" "${INTERSHEET_REFS}" (id 0) (at 283.7483 156.1306 0)
+      (effects (font (size 1.27 1.27)) (justify left) hide)
+    )
+  )
   (global_label "INT_START" (shape input) (at 199.39 119.38 180) (fields_autoplaced)
     (effects (font (size 1.27 1.27)) (justify right))
@@
     )
   )
-  (global_label "~{Fetch_Status}" (shape output) (at 269.24 157.48 0) (fields_autoplaced)
+  (global_label "~{Fetch_Status}" (shape output) (at 269.24 153.67 0) (fields_autoplaced)
     (effects (font (size 1.27 1.27)) (justify left))
-    (property "Intersheet References" "${INTERSHEET_REFS}" (id 0) (at 283.7483 157.4006 0)
+    (property "Intersheet References" "${INTERSHEET_REFS}" (id 0) (at 283.7483 153.5906 0)
       (effects (font (size 1.27 1.27)) (justify left) hide)
     )
   )
-  (global_label "~{SP_INC_RET->}" (shape input) (at 166.37 40.64 180) (fields_autoplaced)
-    (effects (font (size 1.27 1.27)) (justify right))
-    (property "Intersheet References" "${INTERSHEET_REFS}" (id 0) (at 149.8055 40.5606 0)
+  (global_label "~{SP_INC_RET->}" (shape input) (at 166.37 59.69 180) (fields_autoplaced)
+    (effects (font (size 1.27 1.27)) (justify right))
+    (property "Intersheet References" "${INTERSHEET_REFS}" (id 0) (at 149.8055 59.6106 0)
       (effects (font (size 1.27 1.27)) (justify right) hide)
     )
@@
     )
   )
-  (global_label "~{SP_DEC_PUSH->}" (shape input) (at 166.37 59.69 180) (fields_autoplaced)
-    (effects (font (size 1.27 1.27)) (justify right))
-    (property "Intersheet References" "${INTERSHEET_REFS}" (id 0) (at 147.5679 59.6106 0)
-      (effects (font (size 1.27 1.27)) (justify right) hide)
-    )
+  (global_label "~{SP_DEC_PUSH->}" (shape input) (at 166.37 40.64 180) (fields_autoplaced)
+    (effects (font (size 1.27 1.27)) (justify right))
+    (property "Intersheet References" "${INTERSHEET_REFS}" (id 0) (at 147.5679 40.5606 0)
+      (effects (font (size 1.27 1.27)) (justify right) hide)
+    )
