File: nlp-16a/Hardware/ID_interface/3word.kicad_sch (KiCad schematic)
At the start: 16 parts

Commit message: 命令デコーダインターフェイスだいたい完了！！
Parts:
- gave numbers to parts that had none: 4
Connections:
- net 3word: now also U14.8; no longer U13.3
- net GND: now also U12.4, U12.5; no longer U14.1, U14.2
- net RA2_0: now also U12.2; no longer U13.2
- net RA2_1: now also U12.1; no longer U13.1
- net RA2_2: now also U11.12, U11.13; no longer U11.1, U11.2
- net RA3_2: now also U13.12, U13.13; no longer U12.1, U12.2
- net RA3_3: now also U13.1, U13.2; no longer U12.1, U12.2
- net at U11.3: now also U11.4; no longer U11.1
- net at U12.3: now also U12.12, U12.13; no longer U12.1
- new net: U12.10, U12.11
- new net: U12.8, U14.10
- new net: U11.8, U12.9
- new net: U14.12, U14.13, U14.3
- new net: U11.11, U11.5
- new net: U11.10, U11.6, U11.9
- new net: U13.3, U13.4
- new net: U13.11, U13.5
- new net: U13.10, U13.6, U13.9
- new net: U14.6, U14.9
- new net: U14.11, U14.5
- new net: U13.8, U14.4
Other:
- moved on the sheet: U12A, U12B, U12C, U12D, U13A, U13B, U13C, U13D, U14C
