File: nlp-16a/Hardware/ID_interface/A_B_Select.kicad_sch (KiCad schematic)
At the start: 13 parts

Commit message: 命令デコーダインターフェイスだいたい完了！！
Parts:
- added U?: CD74HC00, Package_DIP:DIP-14_W7.62mm, symbol CD74HCxx:CD74HC00
Connections:
- net GND: now also U?.7 (GND)
- net VCC: now also U?.14 (VCC)
- net BUS_A/~{Y}: now reaches U?.1, U?.10, U?.13, U?.2, U?.2, U?.5
Changed lines of the file:
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@@
   (junction (at 144.78 96.52) (diameter 0) (color 0 0 0 0)
   )
+  (junction (at 123.19 144.78) (diameter 0) (color 0 0 0 0)
+  )
   (junction (at 144.78 129.54) (diameter 0) (color 0 0 0 0)
   )
@@
   )
   (wire (pts (xy 142.24 110.49) (xy 142.24 115.57))
+    (stroke (width 0) (type default) (color 0 0 0 0))
+  )
+  (wire (pts (xy 85.09 144.78) (xy 123.19 144.78))
     (stroke (width 0) (type default) (color 0 0 0 0))
   )
@@
     (property "Intersheet References" "${INTERSHEET_REFS}" (id 0) (at 228.2917 140.8906 0)
       (effects (font (size 1.27 1.27)) (justify left) hide)
+    )
+  )
+  (global_label "BUS_A{slash}~{Y}" (shape input) (at 85.09 144.78 180) (fields_autoplaced)
+    (effects (font (size 1.27 1.27)) (justify right))
+    (property "Intersheet References" "${INTERSHEET_REFS}" (id 0) (at 74.3917 144.7006 0)
+      (effects (font (size 1.27 1.27)) (justify right) hide)
     )
   )
@@
     (pin "14")
     (pin "7")
+    (pin "1")
+    (pin "2")
+    (pin "3")
+    (pin "4")
+    (pin "5")
+    (pin "6")
+    (pin "10")
+    (pin "8")
+    (pin "9")
+    (pin "11")
+    (pin "12")
+    (pin "13")
+  )
+  (symbol (lib_id "CD74HCxx:CD74HC00") (at 133.35 161.29 0) (unit 2)
+    (in_bom yes) (on_board yes) (fields_autoplaced)
+    (property "Reference" "U?" (id 0) (at 133.35 152.4 0))
+    (property "Value" "CD74HC00" (id 1) (at 133.35 154.94 0))
+    (property "Footprint" "Package_DIP:DIP-14_W7.62mm" (id 2) (at 128.27 161.29 0)
+      (effects (font (size 1.27 1.27)) hide)
+    )
+    (property "Datasheet" "" (id 3) (at 128.27 161.29 0))
+    (pin "14")
+    (pin "7")
