File: nlp-16a/Hardware/ID_interface/A_Y_Select.kicad_sch (KiCad schematic)
At the start: 13 parts

Commit message: 命令デコーダインターフェイスだいたい完了！！
Connections:
- net BUS_A/~{B}: now reaches U?.1, U?.10, U?.13, U?.2, U?.2, U?.5
Changed lines of the file:
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@@
   (junction (at 125.73 135.89) (diameter 0) (color 0 0 0 0)
   )
+  (junction (at 125.73 151.13) (diameter 0) (color 0 0 0 0)
+  )
   (junction (at 147.32 119.38) (diameter 0) (color 0 0 0 0)
   )
@@
   )
   (wire (pts (xy 147.32 102.87) (xy 147.32 119.38))
+    (stroke (width 0) (type default) (color 0 0 0 0))
+  )
+  (wire (pts (xy 87.63 151.13) (xy 125.73 151.13))
     (stroke (width 0) (type default) (color 0 0 0 0))
   )
@@
       (effects (font (size 1.27 1.27)) (justify right) hide)
     )
+  )
+  (global_label "BUS_A{slash}~{B}" (shape input) (at 87.63 151.13 180) (fields_autoplaced)
+    (effects (font (size 1.27 1.27)) (justify right))
+    (property "Intersheet References" "${INTERSHEET_REFS}" (id 0) (at 76.7502 151.0506 0)
+      (effects (font (size 1.27 1.27)) (justify right) hide)
+    )
