File: nlp-16a/Hardware/ID_interface/Seed_pluse.kicad_sch (KiCad schematic)
At the start: 11 parts

Commit message: 命令デコーダとの配線方法を変更
Parts:
- added U?: CD74HC00, Package_DIP:DIP-14_W7.62mm, symbol CD74HCxx:CD74HC00
Connections:
- net GND: now also U?.1, U?.2, U?.7 (GND)
- net VCC: now also U?.14 (VCC)
- no-connect marks 0 -> 1
Changed lines of the file:
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@@
   (junction (at 125.6584 101.6) (diameter 0) (color 0 0 0 0)
   )
+  (junction (at 64.77 135.89) (diameter 0) (color 0 0 0 0)
+  )
   (junction (at 62.23 99.06) (diameter 0) (color 0 0 0 0)
   )
@@
   (junction (at 179.07 107.95) (diameter 0) (color 0 0 0 0)
   )
+  (no_connect (at 80.01 133.35))
   (wire (pts (xy 149.7884 107.95) (xy 149.7884 118.11))
     (stroke (width 0) (type default) (color 0 0 0 0))
@@
     (stroke (width 0) (type default) (color 0 0 0 0))
   )
+  (wire (pts (xy 64.77 130.81) (xy 64.77 135.89))
+    (stroke (width 0) (type default) (color 0 0 0 0))
+  )
   (wire (pts (xy 60.96 123.19) (xy 60.96 120.65))
     (stroke (width 0) (type default) (color 0 0 0 0))
@@
   )
   (wire (pts (xy 62.23 99.06) (xy 64.77 99.06))
+    (stroke (width 0) (type default) (color 0 0 0 0))
+  )
+  (wire (pts (xy 64.77 135.89) (xy 64.77 139.7))
     (stroke (width 0) (type default) (color 0 0 0 0))
   )
@@
       (effects (font (size 1.27 1.27)) (justify right) hide)
     )
+  )
+  (symbol (lib_id "CD74HCxx:CD74HC00") (at 72.39 133.35 0) (unit 1)
+    (in_bom yes) (on_board yes) (fields_autoplaced)
+    (property "Reference" "U?" (id 0) (at 72.39 124.46 0))
+    (property "Value" "CD74HC00" (id 1) (at 72.39 127 0))
+    (property "Footprint" "Package_DIP:DIP-14_W7.62mm" (id 2) (at 67.31 133.35 0)
+      (effects (font (size 1.27 1.27)) hide)
+    )
+    (property "Datasheet" "" (id 3) (at 67.31 133.35 0))
+    (pin "14")
+    (pin "7")
+    (pin "1")
+    (pin "2")
+    (pin "3")
+    (pin "4")
+    (pin "5")
+    (pin "6")
+    (pin "10")
+    (pin "8")
+    (pin "9")
+    (pin "11")
+    (pin "12")
+    (pin "13")
   )
   (symbol (lib_id "CD74HCxx:CD74HC00") (at 72.39 101.6 0) (unit 1)
@@
     (pin "13")
   )
+  (symbol (lib_id "power:GND") (at 64.77 139.7 0) (unit 1)
+    (in_bom yes) (on_board yes) (fields_autoplaced)
+    (property "Reference" "#PWR?" (id 0) (at 64.77 146.05 0)
+      (effects (font (size 1.27 1.27)) hide)
+    )
+    (property "Value" "GND" (id 1) (at 64.77 144.78 0))
+    (property "Footprint" "" (id 2) (at 64.77 139.7 0)
+      (effects (font (size 1.27 1.27)) hide)
+    )
+    (property "Datasheet" "" (id 3) (at 64.77 139.7 0)
+      (effects (font (size 1.27 1.27)) hide)
+    )
+    (pin "1")
+  )
   (symbol (lib_id "CD74HCxx:CD74HC00") (at 189.23 101.6 0) (unit 1)

Commit message: 命令デコーダインターフェイスだいたい完了！！
Parts:
- gave numbers to parts that had none: 3
Connections:
- net GND: now also U1.12, U1.13; no longer U1.1, U1.2
- net at U1.3: now also U1.4; no longer U1.2
- net phi2_2: now reaches U2.1
- net phi2_2: now also U2.5; no longer U1.3
- net phi1_2: now reaches U3.1
- net phi1_2: now also U3.5
- removed net Seed_pluse: U3.1, U3.3
- net phi1: no longer names the net of U2.2
- net phi1: now also U1.8; no longer U2.2
- net phi2: no longer names the net of U3.2
- net phi2: now also U2.13, U2.8; no longer U3.2
- removed net ~RS: U1.1, U1.1
- new net: U1.1, U1.6, U1.9
- new net: U3.10, U3.11
- new net: U3.12, U3.3, U3.4
- new net: U3.6, U3.9
- new net: U2.10, U2.11
- new net: U2.12, U2.3, U2.4
- new net: U2.6, U2.9
- new net ~{RS}: U1.10, U1.5
- new net ~{Seed_pluse}: U1.2, U3.13, U3.8
Other:
- moved on the sheet: U1D
