File: nlp-16a/Hardware/alu_c/ALUv6.kicad_sch (KiCad schematic)
At the start: 15 parts, among them U1 CD74HC00, U2 CD74HC00, U3 CD74HC00, U4 CD74HC00, U5 CD74HC00, U6 CD74HC00, U7 CD74HC00

Commit message: ALU エラッタ修正版
Connections:
- net B_sign: now reaches U5.2, U6.11, U6.4
Changed lines of the file:
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@@
   (junction (at 161.29 54.61) (diameter 0) (color 0 0 0 0)
+  )
+  (junction (at 148.59 62.23) (diameter 0) (color 0 0 0 0)
   )
   (junction (at 199.39 81.28) (diameter 0) (color 0 0 0 0)
@@
     (stroke (width 0) (type default) (color 0 0 0 0))
   )
-  (wire (pts (xy 143.51 62.23) (xy 200.66 62.23))
+  (wire (pts (xy 143.51 62.23) (xy 148.59 62.23))
     (stroke (width 0) (type default) (color 0 0 0 0))
   )
@@
     (stroke (width 0) (type default) (color 0 0 0 0))
   )
+  (wire (pts (xy 148.59 69.85) (xy 148.59 62.23))
+    (stroke (width 0) (type default) (color 0 0 0 0))
+  )
   (wire (pts (xy 158.75 109.22) (xy 157.48 109.22))
     (stroke (width 0) (type default) (color 0 0 0 0))
@@
     (stroke (width 0) (type default) (color 0 0 0 0))
   )
+  (wire (pts (xy 148.59 62.23) (xy 200.66 62.23))
+    (stroke (width 0) (type default) (color 0 0 0 0))
+  )
   (wire (pts (xy 92.71 64.77) (xy 91.44 64.77))
     (stroke (width 0) (type default) (color 0 0 0 0))
@@
   )
   (wire (pts (xy 123.19 93.98) (xy 121.92 93.98))
+    (stroke (width 0) (type default) (color 0 0 0 0))
+  )
+  (wire (pts (xy 151.13 69.85) (xy 148.59 69.85))
     (stroke (width 0) (type default) (color 0 0 0 0))
   )
@@
     (effects (font (size 1.27 1.27)) (justify right))
   )
+  (hierarchical_label "B_sign" (shape output) (at 151.13 69.85 0)
+    (effects (font (size 1.27 1.27)) (justify left))
+  )
   (hierarchical_label "carry_out" (shape output) (at 242.57 96.52 0)
