File: nlp-16a/Hardware/alu_c/alu_c.kicad_sch (KiCad schematic)
At the start: 53 parts, among them J1 Conn_02x10_Counter_Clockwise, J2 Conn_02x10_Counter_Clockwise, J3 Conn_02x10_Counter_Clockwise, J4 Conn_02x10_Counter_Clockwise, J5 Screw_Terminal_01x02, U57 CD74HC00, U58 CD74HC00, U59 CD74HC00, U60 CD74HC00

Commit message: ALU エラッタ修正版
Connections:
- net B7: no longer J4.5 (Pin_5)
- new net B_sign: J4.5 (Pin_5)
- no-connect marks 7 -> 14
Other:
- sheet ALUv7-No.1 ports: added B_sign; removed none
- sheet ALUv7-No.2 ports: added B_sign; removed none
- sheet ALUv7-No.3 ports: added B_sign; removed none
- sheet ALUv7-No.4 ports: added B_sign; removed none
- sheet ALUv7-No.5 ports: added B_sign; removed none
- sheet ALUv7-No.6 ports: added B_sign; removed none
- sheet ALUv7-No.7 ports: added B_sign; removed none
- sheet ALUv7-No.8 ports: added B_sign; removed none
- moved on the sheet: U57A, U57B, U57C, U57D
