File: nlp-16a/Hardware/alu_ctrl/ALU_Ctrl_Dec.kicad_sch (KiCad schematic)
At the start: 9 parts, among them U19 CD74HC00, U20 CD74HC00, U21 CD74HC00, U22 CD74HC00, U23 CD74HC00, U24 CD74HC00, U25 CD74HC00, U26 CD74HC00, U27 CD74HC00

Commit message: 修正はしていないがkicadで開いたら謎に変更が入った
Other:
- note added: "1,2入れ替え"
Changed lines of the file:
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@@
+    (stroke (width 0) (type default) (color 0 0 0 0))
+  )
+  (polyline (pts (xy 38.1 58.42) (xy 38.1 82.55))
     (stroke (width 0) (type default) (color 0 0 0 0))
   )
@@
     (effects (font (size 1.27 1.27)) (justify left bottom))
   )
+  (text "1,2入れ替え" (at 38.1 62.23 0)
+    (effects (font (size 1.27 1.27)) (justify left bottom))
+  )

Commit message: ALU制御 エラッタ修正版
Parts:
- added U12: CD74HC00, Package_DIP:DIP-14_W7.62mm, symbol CD74HCxx:CD74HC00
Connections:
- net Ctrl2: now also U25.9; no longer U26.1
- net Ctrl8: now also U12.10, U12.9; no longer U23.1, U23.2
- net GND: now also U12.7 (GND)
- net VCC: now also U12.14 (VCC)
- net at U25.6: now also U23.1, U23.2; no longer U25.9
- net at U23.4: now also U12.8; no longer U23.3
- net ~C0 renamed ~{C0}
- net ~C1 renamed ~{C1}
- net ~C2 renamed ~{C2}
- net ~C3 renamed ~{C3}
- new net: U23.3, U26.1
Other:
- note added: "12Cと23Aを交換"
- note removed: "1,2入れ替え"
- note removed: "25,22"
- moved on the sheet: U20B, U22B, U22C, U23A, U25B, U25C, U26A, U26D
