File: nlp-16a/Hardware/BUS_terminator/IO_port.kicad_sch (KiCad schematic)
At the start: 18 parts, among them U1 CD74HC00, U10 CD74HC245, U11 CD74HC00, U12 CD74HC00, U2 CD74HC00, U3 CD74HC00, U4 CD74HC00, U5 CD74HC00, U6 CD74HC00, U7 CD74HC00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

Commit message: アキュムレータ更新
Parts:
- removed U10, U9: CD74HC245, Package_DIP:DIP-20_W7.62mm, symbol CD74HCXX:CD74HC245
- added U10, U9: 74HCT541, Package_DIP:DIP-20_W7.62mm, symbol 74xx:74HCT541
Connections:
- net GND: now also U10.1 (G1), U10.10 (GND), U9.1 (G1), U9.10 (GND)
- net IN0: now also U10.9 (A7)
- net IN1: now also U10.8 (A6)
- net IN10: now also U9.7 (A5)
- net IN11: now also U9.6 (A4)
- net IN12: now also U9.5 (A3)
- net IN13: now also U9.4 (A2)
- net IN14: now also U9.3 (A1)
- net IN15: now also U9.2 (A0)
- net IN2: now also U10.7 (A5)
- net IN3: now also U10.6 (A4)
- net IN4: now also U10.5 (A3)
- net IN5: now also U10.4 (A2)
- net IN6: now also U10.3 (A1)
- net IN7: now also U10.2 (A0)
- net IN8: now also U9.9 (A7)
- net IN9: now also U9.8 (A6)
- net IO_BUS0: now also U10.11 (Y7)
- net IO_BUS1: now also U10.12 (Y6)
- net IO_BUS10: now also U9.13 (Y5)
- net IO_BUS11: now also U9.14 (Y4)
- net IO_BUS12: now also U9.15 (Y3)
- net IO_BUS13: now also U9.16 (Y2)
- net IO_BUS14: now also U9.17 (Y1)
- net IO_BUS15: now also U9.18 (Y0)
- net IO_BUS2: now also U10.13 (Y5)
- net IO_BUS3: now also U10.14 (Y4)
- net IO_BUS4: now also U10.15 (Y3)
- net IO_BUS5: now also U10.16 (Y2)
- net IO_BUS6: now also U10.17 (Y1)
- net IO_BUS7: now also U10.18 (Y0)
- net IO_BUS8: now also U9.11 (Y7)
- net IO_BUS9: now also U9.12 (Y6)
- net VCC: now also U10.20 (VCC), U9.20 (VCC)
- net at D3.1 (K), U12.11: now also U10.19 (G2), U9.19 (G2)
Other:
- moved on the sheet: D3, R19, RN1, RN2

Commit message: バスターミネータのDMA機能は不要と判断したので削除．必要ならば外部回路で実現するように
Parts:
- renumbered D3 to D2, D2 to D3, R19 to R18, R18 to R19
Connections:
- net A_SEL: now also U12.4
- net GND: no longer U12.10, U12.4, U12.5, U12.9
- net Y_SEL: now also U12.10
- net Data_Correction: now reaches U12.3, U5.2, U5.5, U6.2, U6.5, U7.2, U7.5, U8.2, U8.5
- net WR_CLK: now reaches U12.8
- net RD_CLK: now reaches U12.6
- net Correction renamed BUS_Correction
- new net phi1: U12.5
- new net phi2: U12.9
- no-connect marks 2 -> 0
Other:
- moved on the sheet: U12B, U12C

Commit message: v1.1全ガーバーを更新
Connections:
- net at U11.12, U11.13, U11.3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: now also D2.1 (K); no longer D3.1 (K)
- net at U10.19 (G2), U12.11, U9.19 (G2): now also D3.1 (K); no longer D2.1 (K)
Other:
- moved on the sheet: D2, D3, R18, R19
Changed lines of the file:
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@@
     (stroke (width 0) (type default) (color 0 0 0 0))
   )
-  (wire (pts (xy 118.11 154.94) (xy 123.19 154.94))
+  (wire (pts (xy 237.49 162.56) (xy 240.03 162.56))
     (stroke (width 0) (type default) (color 0 0 0 0))
   )
@@
     (stroke (width 0) (type default) (color 0 0 0 0))
   )
+  (wire (pts (xy 123.19 146.05) (xy 123.19 147.32))
+    (stroke (width 0) (type default) (color 0 0 0 0))
+  )
   (wire (pts (xy 96.52 104.14) (xy 101.6 104.14))
     (stroke (width 0) (type default) (color 0 0 0 0))
@@
     (stroke (width 0) (type default) (color 0 0 0 0))
   )
-  (wire (pts (xy 107.95 154.94) (xy 110.49 154.94))
-    (stroke (width 0) (type default) (color 0 0 0 0))
-  )
   (bus (pts (xy 132.08 15.24) (xy 205.74 15.24))
     (stroke (width 0) (type default) (color 0 0 0 0))
@@
     (stroke (width 0) (type default) (color 0 0 0 0))
   )
+  (wire (pts (xy 107.95 154.94) (xy 111.76 154.94))
+    (stroke (width 0) (type default) (color 0 0 0 0))
+  )
   (bus (pts (xy 205.74 99.06) (xy 205.74 114.3))
     (stroke (width 0) (type default) (color 0 0 0 0))
@@
     (stroke (width 0) (type default) (color 0 0 0 0))
   )
-  (wire (pts (xy 237.49 162.56) (xy 240.03 162.56))
+  (wire (pts (xy 119.38 154.94) (xy 123.19 154.94))
     (stroke (width 0) (type default) (color 0 0 0 0))
   )
@@
   )
   (wire (pts (xy 77.47 106.68) (xy 81.28 106.68))
-    (stroke (width 0) (type default) (color 0 0 0 0))
-  )
-  (wire (pts (xy 123.19 154.94) (xy 123.19 153.67))
     (stroke (width 0) (type default) (color 0 0 0 0))
   )
@@
     (pin "13")
   )
-  (symbol (lib_id "Device:R") (at 240.03 158.75 0) (unit 1)
-    (in_bom yes) (on_board yes) (fields_autoplaced)
-    (property "Reference" "R18" (id 0) (at 242.57 157.4799 0)
+  (symbol (lib_id "Device:R") (at 123.19 151.13 0) (unit 1)
+    (in_bom yes) (on_board yes) (fields_autoplaced)
+    (property "Reference" "R18" (id 0) (at 125.73 149.8599 0)
       (effects (font (size 1.27 1.27)) (justify left))
     )
-    (property "Value" "R" (id 1) (at 242.57 160.0199 0)
+    (property "Value" "R" (id 1) (at 125.73 152.3999 0)
       (effects (font (size 1.27 1.27)) (justify left))
     )
-    (property "Footprint" "Resistor_SMD:R_0603_1608Metric_Pad0.98x0.95mm_HandSolder" (id 2) (at 238.252 158.75 90)
-      (effects (font (size 1.27 1.27)) hide)
-    )
-    (property "Datasheet" "~" (id 3) (at 240.03 158.75 0)
+    (property "Footprint" "Resistor_SMD:R_0603_1608Metric_Pad0.98x0.95mm_HandSolder" (id 2) (at 121.412 151.13 90)
+      (effects (font (size 1.27 1.27)) hide)
+    )
+    (property "Datasheet" "~" (id 3) (at 123.19 151.13 0)
       (effects (font (size 1.27 1.27)) hide)
     )
@@
     (pin "1")
   )
-  (symbol (lib_id "Device:R") (at 123.19 149.86 0) (unit 1)
-    (in_bom yes) (on_board yes) (fields_autoplaced)
-    (property "Reference" "R19" (id 0) (at 125.73 148.5899 0)
+  (symbol (lib_id "Device:R") (at 240.03 158.75 0) (unit 1)
+    (in_bom yes) (on_board yes) (fields_autoplaced)
+    (property "Reference" "R19" (id 0) (at 242.57 157.4799 0)
       (effects (font (size 1.27 1.27)) (justify left))
     )
-    (property "Value" "R" (id 1) (at 125.73 151.1299 0)
+    (property "Value" "R" (id 1) (at 242.57 160.0199 0)
       (effects (font (size 1.27 1.27)) (justify left))
     )
-    (property "Footprint" "Resistor_SMD:R_0603_1608Metric_Pad0.98x0.95mm_HandSolder" (id 2) (at 121.412 149.86 90)
-      (effects (font (size 1.27 1.27)) hide)
-    )
-    (property "Datasheet" "~" (id 3) (at 123.19 149.86 0)
+    (property "Footprint" "Resistor_SMD:R_0603_1608Metric_Pad0.98x0.95mm_HandSolder" (id 2) (at 238.252 158.75 90)
+      (effects (font (size 1.27 1.27)) hide)
+    )
+    (property "Datasheet" "~" (id 3) (at 240.03 158.75 0)
       (effects (font (size 1.27 1.27)) hide)
     )
@@
     (pin "1")
   )
-  (symbol (lib_id "Device:LED") (at 114.3 154.94 0) (unit 1)
+  (symbol (lib_id "Device:LED") (at 233.68 162.56 0) (unit 1)
     (in_bom yes) (on_board yes)
-    (property "Reference" "D3" (id 0) (at 111.76 152.4 0))
-    (property "Value" "LED" (id 1) (at 116.84 152.4 0))
-    (property "Footprint" "LED_THT:LED_D3.0mm" (id 2) (at 114.3 154.94 0)
-      (effects (font (size 1.27 1.27)) hide)
-    )
-    (property "Datasheet" "~" (id 3) (at 114.3 154.94 0)
+    (property "Reference" "D3" (id 0) (at 231.14 160.02 0))
+    (property "Value" "LED" (id 1) (at 236.22 160.02 0))
+    (property "Footprint" "LED_THT:LED_D3.0mm" (id 2) (at 233.68 162.56 0)
+      (effects (font (size 1.27 1.27)) hide)
+    )
+    (property "Datasheet" "~" (id 3) (at 233.68 162.56 0)
       (effects (font (size 1.27 1.27)) hide)
     )
@@
     (pin "13")
   )
-  (symbol (lib_id "Device:LED") (at 233.68 162.56 0) (unit 1)
+  (symbol (lib_id "Device:LED") (at 115.57 154.94 0) (unit 1)
     (in_bom yes) (on_board yes)
-    (property "Reference" "D2" (id 0) (at 231.14 160.02 0))
-    (property "Value" "LED" (id 1) (at 236.22 160.02 0))
-    (property "Footprint" "LED_THT:LED_D3.0mm" (id 2) (at 233.68 162.56 0)
-      (effects (font (size 1.27 1.27)) hide)
-    )
-    (property "Datasheet" "~" (id 3) (at 233.68 162.56 0)
-      (effects (font (size 1.27 1.27)) hide)
-    )
+    (property "Reference" "D2" (id 0) (at 113.03 152.4 0))
+    (property "Value" "LED" (id 1) (at 118.11 152.4 0))
+    (property "Footprint" "LED_THT:LED_D3.0mm" (id 2) (at 115.57 154.94 0)
+      (effects (font (size 1.27 1.27)) hide)
+    )
+    (property "Datasheet" "~" (id 3) (at 115.57 154.94 0)
+      (effects (font (size 1.27 1.27)) hide)
+    )
