File: nlp-16a/Hardware/RAM_board/RAM_board.kicad_sch (KiCad schematic)
At the start: 23 parts, among them J1 Conn_02x10_Odd_Even, J2 Conn_02x20_Odd_Even, J3 Conn_02x10_Odd_Even, J4 Conn_02x20_Odd_Even, J5 Conn_02x10_Odd_Even, J6 Screw_Terminal_01x02, SW1 SW_Push, U1 TC551001, U2 TC551001, U3 74LS32

Commit message: RAMボードの部品の値を修正
Parts:
- U3: value 74LS32 -> 74LS08
Changed lines of the file:
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@@
     (in_bom yes) (on_board yes) (fields_autoplaced)
     (property "Reference" "U3" (id 0) (at 57.15 143.51 0))
-    (property "Value" "74LS32" (id 1) (at 57.15 146.05 0))
+    (property "Value" "74LS08" (id 1) (at 57.15 146.05 0))
     (property "Footprint" "Package_DIP:DIP-14_W7.62mm" (id 2) (at 57.15 152.4 0)
       (effects (font (size 1.27 1.27)) hide)
@@
     (in_bom yes) (on_board yes) (fields_autoplaced)
     (property "Reference" "U3" (id 0) (at 57.15 173.99 0))
-    (property "Value" "74LS32" (id 1) (at 57.15 176.53 0))
+    (property "Value" "74LS08" (id 1) (at 57.15 176.53 0))
     (property "Footprint" "Package_DIP:DIP-14_W7.62mm" (id 2) (at 57.15 182.88 0)
       (effects (font (size 1.27 1.27)) hide)
@@
     (in_bom yes) (on_board yes) (fields_autoplaced)
     (property "Reference" "U3" (id 0) (at 57.15 158.75 0))
-    (property "Value" "74LS32" (id 1) (at 57.15 161.29 0))
+    (property "Value" "74LS08" (id 1) (at 57.15 161.29 0))
     (property "Footprint" "Package_DIP:DIP-14_W7.62mm" (id 2) (at 57.15 167.64 0)
       (effects (font (size 1.27 1.27)) hide)
@@
       (effects (font (size 1.27 1.27)) (justify left))
     )
-    (property "Value" "74LS32" (id 1) (at 139.7 170.1799 0)
+    (property "Value" "74LS08" (id 1) (at 139.7 170.1799 0)
       (effects (font (size 1.27 1.27)) (justify left))
     )
@@
     (in_bom yes) (on_board yes) (fields_autoplaced)
     (property "Reference" "U3" (id 0) (at 115.57 160.02 0))
-    (property "Value" "74LS32" (id 1) (at 115.57 162.56 0))
+    (property "Value" "74LS08" (id 1) (at 115.57 162.56 0))
     (property "Footprint" "Package_DIP:DIP-14_W7.62mm" (id 2) (at 115.57 168.91 0)
       (effects (font (size 1.27 1.27)) hide)
@@
     )
     (path "/3e7d310c-5535-4cce-aa20-b6fc2634fff3"
-      (reference "U3") (unit 1) (value "74LS32") (footprint "Package_DIP:DIP-14_W7.62mm")
+      (reference "U3") (unit 1) (value "74LS08") (footprint "Package_DIP:DIP-14_W7.62mm")
     )
     (path "/a035e540-a5c1-4288-8ae3-ecc2a3a9c360"
-      (reference "U3") (unit 2) (value "74LS32") (footprint "Package_DIP:DIP-14_W7.62mm")
+      (reference "U3") (unit 2) (value "74LS08") (footprint "Package_DIP:DIP-14_W7.62mm")
     )
     (path "/f9e82164-5f52-4b9e-9cb9-b77c6fd07812"
-      (reference "U3") (unit 3) (value "74LS32") (footprint "Package_DIP:DIP-14_W7.62mm")
+      (reference "U3") (unit 3) (value "74LS08") (footprint "Package_DIP:DIP-14_W7.62mm")
     )
     (path "/b30367f1-cb8c-4dd5-b2e4-12c42f203505"
-      (reference "U3") (unit 4) (value "74LS32") (footprint "Package_DIP:DIP-14_W7.62mm")
+      (reference "U3") (unit 4) (value "74LS08") (footprint "Package_DIP:DIP-14_W7.62mm")
     )
     (path "/d605225b-f457-4511-aade-cf2517f61129"
-      (reference "U3") (unit 5) (value "74LS32") (footprint "Package_DIP:DIP-14_W7.62mm")
-    )
-  )
+      (reference "U3") (unit 5) (value "74LS08") (footprint "Package_DIP:DIP-14_W7.62mm")
+    )
+  )
